File: X16-Backplane.sch (EAGLE design)
At the start: 8 parts, among them J1 CONN_PXC-8-RA-1778683, J2 CONN_ET60S-D04-3-08-D04-X-R1-S, J3 CONN_HTST-108-04-X-D-RAJ, U1 TRANS_ULN2003AD

Commit message: 9/27/2023
Connections:
- net SPI1 renamed SPI_MOSI
- net SPI2 renamed SPI_MISO
- net SPI3 renamed SPI_SCLK
- net SPI4 renamed SPI_SS/CS
- new net ESC_ID: U$1.12
- new net N$25: U$1.5
- new net N$26: U$1.7
- new net N$4: U$1.8
- new net NRST: U$1.6
- new net SWCLK: U$1.11
- new net SWDIO: U$1.9
- net 3V3: now also U$1.1, U$1.2, U$1.3, U$1.4
- net GND: now also U$1.10
Changed lines of the file:
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@@
 <setting verticaltext="up"/>
 </settings>
-<grid distance="0.1" unitdist="inch" unit="inch" style="lines" multiple="1" display="no" altdistance="0.01" altunitdist="inch" altunit="inch"/>
+<grid distance="50" unitdist="mil" unit="mil" style="lines" multiple="1" display="no" altdistance="5" altunitdist="mil" altunit="mil"/>
 <layers>
 <layer number="1" name="Top" color="4" fill="1" visible="no" active="no"/>
@@
 <label x="246.38" y="91.44" size="1.778" layer="95"/>
 </segment>
+<segment>
+<pinref part="U$1" gate="G$1" pin="10"/>
+<wire x1="159.004" y1="217.17" x2="165.354" y2="217.17" width="0.1524" layer="91"/>
+<label x="165.1" y="217.17" size="1.778" layer="95"/>
+</segment>
 </net>
 <net name="3V3" class="0">
@@
 <label x="43.18" y="53.34" size="1.778" layer="95"/>
 </segment>
-</net>
-<net name="SPI1" class="0">
+<segment>
+<pinref part="U$1" gate="G$1" pin="2"/>
+<wire x1="159.004" y1="227.33" x2="165.1" y2="227.33" width="0.1524" layer="91"/>
+<label x="165.354" y="227.33" size="1.778" layer="95"/>
+</segment>
+<segment>
+<pinref part="U$1" gate="G$1" pin="4"/>
+<wire x1="159.004" y1="224.79" x2="165.1" y2="224.79" width="0.1524" layer="91"/>
+<label x="165.354" y="224.79" size="1.778" layer="95"/>
+</segment>
+<segment>
+<pinref part="U$1" gate="G$1" pin="1"/>
+<wire x1="136.144" y1="227.33" x2="129.794" y2="227.33" width="0.1524" layer="91"/>
+<label x="129.54" y="227.33" size="1.778" layer="95"/>
+</segment>
+<segment>
+<pinref part="U$1" gate="G$1" pin="3"/>
+<wire x1="136.144" y1="224.79" x2="129.794" y2="224.79" width="0.1524" layer="91"/>
+<label x="129.54" y="224.79" size="1.778" layer="95"/>
+</segment>
+</net>
+<net name="SPI_MOSI" class="0">
 <segment>
 <pinref part="J3" gate="A" pin="13"/>
 <wire x1="50.8" y1="50.8" x2="43.18" y2="50.8" width="0.1524" layer="91"/>
-<label x="43.18" y="50.8" size="1.778" layer="95"/>
-</segment>
-</net>
-<net name="SPI2" class="0">
+<label x="43.18" y="50.8" size="1.778" layer="95" rot="R180"/>
+</segment>
+</net>
+<net name="SPI_MISO" class="0">
 <segment>
 <pinref part="J3" gate="A" pin="15"/>
 <wire x1="50.8" y1="48.26" x2="43.18" y2="48.26" width="0.1524" layer="91"/>
-<label x="43.18" y="48.26" size="1.778" layer="95"/>
-</segment>
-</net>
-<net name="SPI3" class="0">
+<label x="43.18" y="48.26" size="1.778" layer="95" rot="R180"/>
+</segment>
+</net>
+<net name="SPI_SCLK" class="0">
 <segment>
 <pinref part="J3" gate="A" pin="14"/>
@@
 </segment>
 </net>
-<net name="SPI4" class="0">
+<net name="SPI_SS/CS" class="0">
 <segment>
 <pinref part="J3" gate="A" pin="16"/>
@@
 </segment>
 </net>
+<net name="NRST" class="0">
+<segment>
+<pinref part="U$1" gate="G$1" pin="6"/>
+<wire x1="159.004" y1="222.25" x2="165.354" y2="222.25" width="0.1524" layer="91"/>
+<label x="165.1" y="222.25" size="1.778" layer="95"/>
+</segment>
+</net>
+<net name="N$4" class="0">
+<segment>
+<pinref part="U$1" gate="G$1" pin="8"/>
+<wire x1="159.004" y1="219.71" x2="165.354" y2="219.71" width="0.1524" layer="91"/>
+</segment>
+</net>
+<net name="ESC_ID" class="0">
+<segment>
+<pinref part="U$1" gate="G$1" pin="12"/>
+<wire x1="159.004" y1="214.63" x2="165.354" y2="214.63" width="0.1524" layer="91"/>
+<label x="165.1" y="214.63" size="1.778" layer="95"/>
+</segment>
+</net>
+<net name="N$25" class="0">
+<segment>
+<pinref part="U$1" gate="G$1" pin="5"/>
+<wire x1="136.144" y1="222.25" x2="129.794" y2="222.25" width="0.1524" layer="91"/>
+</segment>
+</net>
+<net name="N$26" class="0">
+<segment>
+<pinref part="U$1" gate="G$1" pin="7"/>
+<wire x1="136.144" y1="219.71" x2="129.794" y2="219.71" width="0.1524" layer="91"/>
+</segment>
+</net>
+<net name="SWDIO" class="0">
+<segment>
+<pinref part="U$1" gate="G$1" pin="9"/>
+<wire x1="136.144" y1="217.17" x2="129.794" y2="217.17" width="0.1524" layer="91"/>
+<label x="129.54" y="217.17" size="1.778" layer="95" rot="R180"/>
+</segment>
+</net>
+<net name="SWCLK" class="0">
+<segment>
+<pinref part="U$1" gate="G$1" pin="11"/>
+<wire x1="136.144" y1="214.63" x2="129.794" y2="214.63" width="0.1524" layer="91"/>
+<label x="129.54" y="214.63" size="1.778" layer="95" rot="R180"/>
+</segment>
+</net>

Commit message: 09/30/2023
Parts:
- added D1, D2, D3: (no value), SparkFun-LED:LED0603
- added R1, R2, R3: (no value), SparkFun-Resistors:RESISTOR0603
Connections:
- net N$10 renamed PWMA3
- net N$12 renamed PWMB0
- net N$13 renamed PWMB1
- net N$14 renamed PWMB2
- net N$15 renamed PWMB3
- net N$17 renamed PWMC0
- net N$18 renamed PWMC1
- net N$19 renamed PWMC2
- net N$20 renamed PWMC3
- net N$7 renamed PWMA0
- net N$8 renamed PWMA1
- net N$9 renamed PWMA2
- removed net ESC_ID: U$1.12
- removed net N$25: U$1.5
- removed net N$26: U$1.7
- removed net N$4: U$1.8
- removed net SPI_MISO: J3.15
- removed net SPI_MOSI: J3.13
- removed net SPI_SCLK: J3.14
- removed net SPI_SS/CS: J3.16
- new net ALERT1: J2.ALERT1
- new net ALERT2: J2.ALERT2
- new net C2_1: J2.C2_1
- new net C2_2: J2.C2_2
- new net CLK: J2.CLK
- new net DATA: J2.DATA
- new net MISO: J3.15, U$1.7
- new net MOSI: J3.13, U$1.5
- new net N$1: D1.C, R1.2
- new net N$5: D2.C, R2.2
- new net N$8: D3.C, R3.2
- new net SCLK: J3.14, U$1.8
- new net SS/CS: J3.16, U$1.10
- net 12L_GND: now also J2.12L_GND
- net 12V: now also D1.A, D2.A, D3.A, J2.P06, J2.P07, J2.P08, J2.P09, J2.P10
- net 12V_L: now also J2.12V_L
- net 3V3: now also J2.3V3
- net 5V: now also J2.5V
- net GND: now also J2.GND, J2.P01, J2.P02, J2.P03, J2.P04, J2.P05, R1.1, R2.1, R3.1, U$1.12; no longer U$1.10
Other:
- note added: "12V CAPACITORS"
- note added: "12V LED CHECK"
- note added: "3V LED CHECK"
- note added: "5V LED CHECK"

Commit message: 9/30/2023
Parts:
- removed D3: (no value), SparkFun-LED:LED0603
- removed R3: (no value), SparkFun-Resistors:RESISTOR0603
Connections:
- removed net 12L_GND: J2.12L_GND, J3.5
- removed net ALERT1: J2.ALERT1
- removed net ALERT2: J2.ALERT2
- removed net C2_1: J2.C2_1
- removed net C2_2: J2.C2_2
- removed net CLK: J2.CLK
- removed net DATA: J2.DATA
- removed net N$8: D3.C, R3.2
- removed net NRST: U$1.6
- removed net SWDIO: U$1.9
- net 12V: now also J2.P01, J2.P02; no longer D3.A, J2.P06, J2.P07, J2.P08, J2.P09, J2.P10
- net 12V_GND: now also J2.P03, J2.P04
- net 12V_L: no longer J2.12V_L
- net 3V3: no longer J2.3V3, U$1.1, U$1.2, U$1.3, U$1.4
- net 5V: now also J2.P07, J2.P08, U$1.1, U$1.2, U$1.3, U$1.4; no longer J2.5V
- net GND: now also J2.P06; no longer J2.GND, J2.P01, J2.P02, J2.P03, J2.P04, R3.1
Other:
- note removed: "3V LED CHECK"

Commit message: schematic_complete?
Parts:
- J3: value CONN_HTST-108-04-X-D-RAJ -> SAMTEC-HTST-110-04-X-D-RAJ; device X16_Backplane:CONN_HTST-108-04-X-D-RAJ -> SAMTEC-HTST-110-04-X-D-RA:SAMTEC-HTST-110-04-X-D-RAJ
Connections:
- removed net 3V3: J3.11
- removed net GPIO5: J3.10, U1.IN5
- removed net GPIO6: J3.12, U1.IN6
- removed net N$23: U1.OUT7
- removed net N$30: U1.IN7
- removed net SOL5_1: J1.7, U1.OUT5
- removed net SOL6_1: J1.8, U1.OUT6
- removed net SS/CS: J3.16, U$1.10
- removed net SWCLK: U$1.11
- new net CS: J3.20, U$1.11
- new net CTRL: J2.17, J3.7
- new net DGND: J2.18, J3.9
- new net PWM1: U$1.6
- new net PWM2: U$1.8
- new net PWM3: U$1.10
- new net PWM4: U$1.12
- new net SA0: J2.23, J3.19
- new net SA1: J2.22, J3.17
- new net SALERT: J2.20, J3.13
- new net SCL: J2.21, J3.15
- new net SDA: J2.19, J3.11
- net 5V: now also J3.1; no longer J3.7, U$1.2, U$1.4
- net GND: now also J1.7, J1.8, J3.3, U$1.2, U$1.4; no longer J3.9, U$1.12
- net MISO: now also J3.14, U$1.5; no longer J3.15, U$1.7
- net MOSI: now also J3.16, U$1.7; no longer J3.13, U$1.5
- net SCLK: now also J3.18, U$1.9; no longer J3.14, U$1.8

Commit message: 10/14 sch issues fixed
Parts:
- added 12V, 5V, CS, GND, MISO, MOSI, SCLK: TEST-POINT3, SparkFun-Connectors:TEST-POINT3
- added C1, C2, C3: EEE-FT1E561UP, X16_Backplane:EEE-FT1E561UP
- U$1: value CONN_BACKPLANE_ESC_CONTROLLERBKP -> SAMTEC-HTST-110-04-X-D-RAJ; device X16_Backplane:CONN_BACKPLANE_ESC_CONTROLLERBKP -> SAMTEC-HTST-110-04-X-D-RA:SAMTEC-HTST-110-04-X-D-RAJ
Connections:
- removed net N$11: U$2.NC
- removed net N$16: U$3.NC
- removed net N$21: U$4.NC
- removed net PWM1: U$1.6
- removed net PWM2: U$1.8
- removed net PWM3: U$1.10
- removed net PWM4: U$1.12
- net 12V: now also C1.1, C2.1, C3.1; no longer D2.A
- net 12V_GND: now also C1.2, C2.2, C3.2
- net 5V: now also D2.A
- net PWMA0: now also U$1.13
- net PWMA1: now also U$1.15
- net PWMA2: now also U$1.17
- net PWMA3: now also U$1.19
- net PWMB0: now also U$1.6
- net PWMB1: now also U$1.8
- net PWMB2: now also U$1.10
- net PWMB3: now also U$1.12
- net PWMC0: now also U$1.14
- net PWMC1: now also U$1.16
- net PWMC2: now also U$1.18
- net PWMC3: now also U$1.20

Commit message: Update X16-Backplane.sch
Parts:
- renumbered 12V to TP_12V, 5V to TP_5V, CS to TP_CS, GND to TP_GND, MISO to TP_MISO, MOSI to TP_MOSI, SCLK to TP_SCLK, U$1 to J4
Connections:
- net 12V: now also TP_12V.1
- net 5V: now also TP_5V.1
- net CS: now also TP_CS.1
- net GND: now also TP_GND.1
- net MISO: now also TP_MISO.1
- net MOSI: now also TP_MOSI.1
- net SCLK: now also TP_SCLK.1
