File: X16-Backplane1.brd (EAGLE design)
At the start: 160 x 100 mm, 15 parts, among them J1 CONN_PXC-8-RA-1778683, J2 CONN_ET60S-D04-3-08-D04-X-R1-S, J3 SAMTEC-HTST-110-04-X-D-RAJ, J4 SAMTEC-HTST-110-04-X-D-RAJ, U1 TRANS_ULN2003AD

Commit message: Add files via upload
Parts:
- removed J4: SAMTEC-HTST-110-04-X-D-RAJ, X16_Backplane:SAMTEC-HTST-110-04-X-D-RA
- removed U1: TRANS_ULN2003AD, X16_Backplane:16-SOIC
- added J5: SAMTEC-HTST-110-04-X-D-RAJ, X16_Backplane:SAMTEC-HTST-110-04-X-D-RA
- added TP1, TP2, TP3, TP4, TP5, TP6, TP7: TEST-POINT3, SparkFun-Connectors:PAD.03X.03
- added U2: TRANS_ULN2003AD, X16_Backplane:16-SOIC
- moved C2 185.6 mm to (-105.4, -229.9)
- moved C3 185.6 mm to (-105.4, -255.3)
- moved C1 185.6 mm to (-105.4, -204.5)
- moved J3 175.5 mm to (-102.9, -304.8)
- moved U$3 117.3 mm to (1.27, 67.3)
Connections:
- net 12V: now also TP1.1
- net 12V_L: now also U2.9; no longer U1.9
- net 5V: now also J5.1, J5.3, TP2.1; no longer J3.3, J4.1
- net CS: now also J3.20, J5.11, TP7.1; no longer J3.11, J4.20
- net CTRL: now also J3.7; no longer J4.7
- net DGND: now also J3.9; no longer J4.9
- net GND: now also J3.3, J5.2, J5.4, TP3.1, U2.8; no longer J3.2, J3.4, J4.3, U1.8
- net GPIO1: now also J3.2, U2.1; no longer J4.2, U1.1
- net GPIO2: now also J3.4, U2.2; no longer J4.4, U1.2
- net GPIO3: now also J3.6, U2.3; no longer J4.6, U1.3
- net GPIO4: now also J3.8, U2.4; no longer J4.8, U1.4
- net MISO: now also J3.14, J5.5, TP4.1; no longer J3.5, J4.14
- net MOSI: now also J3.16, J5.7, TP5.1; no longer J3.7, J4.16
- net PWMA0: now also J5.13; no longer J3.13
- net PWMA1: now also J5.15; no longer J3.15
- net PWMA2: now also J5.17; no longer J3.17
- net PWMA3: now also J5.19; no longer J3.19
- net PWMB0: now also J5.6; no longer J3.6
- net PWMB1: now also J5.8; no longer J3.8
- net PWMB2: now also J5.10; no longer J3.10
- net PWMB3: now also J5.12; no longer J3.12
- net PWMC0: now also J5.14; no longer J3.14
- net PWMC1: now also J5.16; no longer J3.16
- net PWMC2: now also J5.18; no longer J3.18
- net PWMC3: now also J5.20; no longer J3.20
- net SA0: now also J3.17; no longer J4.17
- net SA1: now also J3.19; no longer J4.19
- net SALERT: now also J3.13; no longer J4.13
- net SCL: now also J3.15; no longer J4.15
- net SCLK: now also J3.18, J5.9, TP6.1; no longer J3.9, J4.18
- net SDA: now also J3.11; no longer J4.11
- net SOL1_1: now also U2.16; no longer U1.16
- net SOL2_1: now also U2.15; no longer U1.15
- net SOL3_1: now also U2.14; no longer U1.14
- net SOL4_1: now also U2.13; no longer U1.13
Other:
- board size 160 x 100 mm -> 139.7 x 110 mm

Commit message: Add files via upload
Parts:
- removed J5: SAMTEC-HTST-110-04-X-D-RAJ, X16_Backplane:SAMTEC-HTST-110-04-X-D-RA
- added J4: CLT-110-01-F-D, X16_Backplane:SAMTEC_CLT-110-01-F-D
- moved J3 322.8 mm to (52.1, -21.6)
- moved U$2 176.4 mm to (50.8, 106.7), turned to 270 degrees
- moved J2 166.7 mm to (11.4, 47.0), flipped to the bottom, turned to 270 degrees
- moved U$1 159.3 mm to (5.08, 106.7), turned to 270 degrees
- moved U$3 101.9 mm to (95.2, 106.7), turned to 270 degrees
- moved U2 2.54 mm to (-121.9, -189.2)
Connections:
- net 5V: now also J4.01, J4.03; no longer J5.1, J5.3
- net CS: now also J4.11; no longer J5.11
- net GND: now also J4.02, J4.04; no longer J5.2, J5.4
- net MISO: now also J4.05; no longer J5.5
- net MOSI: now also J4.07; no longer J5.7
- net PWMA0: now also J4.13; no longer J5.13
- net PWMA1: now also J4.15; no longer J5.15
- net PWMA2: now also J4.17; no longer J5.17
- net PWMA3: now also J4.19; no longer J5.19
- net PWMB0: now also J4.06; no longer J5.6
- net PWMB1: now also J4.08; no longer J5.8
- net PWMB2: now also J4.10; no longer J5.10
- net PWMB3: now also J4.12; no longer J5.12
- net PWMC0: now also J4.14; no longer J5.14
- net PWMC1: now also J4.16; no longer J5.16
- net PWMC2: now also J4.18; no longer J5.18
- net PWMC3: now also J4.20; no longer J5.20
- net SCLK: now also J4.09; no longer J5.9

Commit message: Add files via upload
Parts:
- moved TP7 477.3 mm to (77.5, 104.1), flipped to the bottom, turned to 270 degrees
- moved TP6 473.9 mm to (74.9, 104.1), flipped to the bottom, turned to 270 degrees
- moved TP5 470.6 mm to (72.4, 104.1), flipped to the bottom, turned to 270 degrees
- moved TP4 467.2 mm to (69.8, 104.1), flipped to the bottom, turned to 270 degrees
- moved TP3 463.8 mm to (67.3, 104.1), flipped to the bottom, turned to 270 degrees
- moved TP2 460.5 mm to (64.8, 104.1), flipped to the bottom, turned to 270 degrees
- moved TP1 457.1 mm to (62.2, 104.1), flipped to the bottom, turned to 270 degrees
- moved J4 410.8 mm to (106.7, 10.2)
- moved C3 400.6 mm to (123.2, 73.7)
- moved C2 391.2 mm to (123.2, 87.6)
- moved C1 382.0 mm to (123.2, 101.6)
- moved U2 314.5 mm to (92.7, 40.6), flipped to the bottom
- moved R1 306.5 mm to (10.2, 104.1), flipped to the bottom
- moved R2 294.9 mm to (10.2, 87.6), flipped to the bottom
- moved D1 293.9 mm to (10.2, 100.3), flipped to the bottom
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
Commit message: Add files via upload
Parts:
- moved J3 96.3 mm to (69.8, 111.8), flipped to the bottom
- moved J4 83.0 mm to (73.7, 86.4), flipped to the bottom, turned to 270 degrees
- moved TP1 35.6 mm to (97.8, 102.9)
- moved TP2 35.6 mm to (100.3, 102.9)
- moved TP3 35.6 mm to (102.9, 102.9)
- moved TP4 35.6 mm to (105.4, 102.9)
- moved TP5 35.6 mm to (108.0, 102.9)
- moved TP7 35.6 mm to (113.0, 102.9)
- moved TP6 35.6 mm to (110.5, 102.9)
- moved U2 31.9 mm to (124.5, 38.1)
- moved J1 26.7 mm to (100.3, 31.8)
- moved R2 19.4 mm to (20.3, 104.1)
- moved D2 13.7 mm to (21.6, 100.3)
- moved J2 6.35 mm to (11.4, 53.3)
Routing:
- net 5V: track 0.00 -> 64.8 mm
- net GND: track 0.00 -> 48.5 mm
- net N$5: track 0.00 -> 4.34 mm
- net N$2: track 0.00 -> 3.81 mm
- added copper zone on layer 1, net 12V
- added copper zone on layer 1, net GND

Commit message: Add files via upload
Connections:
- net 12V: now also C1.1, C2.1, C3.1; no longer C1.2, C2.2, C3.2
- net 12V_GND: no longer C1.1, C2.1, C3.1
- net GND: now also C1.2, C2.2, C3.2; no longer J1.7, J1.8, U2.8

Commit message: Add files via upload
Parts:
- moved TP1 27.7 mm to (125.5, 102.4)
- moved TP3 15.0 mm to (117.9, 102.1)
- moved C1 13.8 mm to (121.9, 87.9), flipped to the bottom
- moved C2 12.5 mm to (121.9, 75.2), flipped to the bottom
- moved C3 11.0 mm to (121.9, 62.7), flipped to the bottom
- moved TP5 9.91 mm to (98.8, 106.7)
- moved J4 7.28 mm to (70.1, 80.0)
- moved TP7 6.25 mm to (107.4, 100.1)
- moved TP2 6.18 mm to (106.4, 103.9)
- moved U2 5.79 mm to (118.9, 39.6)
- moved TP6 4.32 mm to (110.5, 98.6)
- moved TP4 3.61 mm to (102.6, 105.2)
- moved J1 1.80 mm to (98.6, 32.0)
Connections:
- new net GPIO5: J3.9, U2.5
- new net GPIO6: J3.5, U2.6
- new net GPIO7: J3.10, U2.7
- new net GPIO8: J3.12
- new net SOL5_1: J1.4, U2.12
- new net SOL6_1: J1.3, U2.11
- new net SOL7_1: U2.10
- net DGND: no longer J3.9
- net SOL1_1: now also J1.8; no longer J1.3
- net SOL2_1: now also J1.7; no longer J1.4
- net SOL3_1: now also J1.6; no longer J1.5
- net SOL4_1: now also J1.5; no longer J1.6
Routing:
- net GND: track 48.5 -> 79.9 mm
- net 12V: track 0.00 -> 30.0 mm
- net 12V_L: track 0.00 -> 14.7 mm
- net SOL1_1: track 0.00 -> 14.5 mm
- net SOL2_1: track 0.00 -> 13.3 mm
- net SOL3_1: track 0.00 -> 12.7 mm
- net SOL4_1: track 0.00 -> 12.2 mm
- net SOL5_1: track 0.00 -> 11.7 mm
- net SOL6_1: track 0.00 -> 11.2 mm

Commit message: Add files via upload
Parts:
- moved J1 74.8 mm to (105.9, 106.4), turned to 180 degrees
- moved C3 64.4 mm to (62.0, 39.1), turned to 90 degrees
- moved C1 59.9 mm to (87.1, 39.1), turned to 90 degrees
- moved C2 59.4 mm to (74.7, 39.1), turned to 90 degrees
- moved U2 51.9 mm to (116.8, 91.4), turned to 90 degrees
- moved D1 44.8 mm to (45.7, 73.2)
- moved D2 44.8 mm to (57.1, 73.2)
- moved R1 44.8 mm to (45.7, 77.0)
- moved R2 44.8 mm to (55.9, 77.0)
- moved J3 41.7 mm to (28.2, 111.3)
- moved TP1 38.4 mm to (87.1, 103.1)
- moved TP3 38.4 mm to (79.5, 102.9)
- moved TP4 38.4 mm to (64.3, 105.9)
- moved TP2 34.3 mm to (72.1, 104.4)
- moved TP5 30.8 mm to (68.1, 105.7)
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Connections:
- removed net DGND: J2.18
- net GND: now also J2.18, U2.8
Routing:
- net 5V: track 64.8 -> 97.0 mm
- net GND: track 79.9 -> 48.5 mm
- net 12V: track 30.0 -> 0.00 mm
- net 12V_L: track 14.7 -> 0.00 mm
- net SOL1_1: track 14.5 -> 0.00 mm
- net SOL2_1: track 13.3 -> 0.00 mm
- net SOL3_1: track 12.7 -> 0.00 mm
- net SOL4_1: track 12.2 -> 0.00 mm
- net SOL5_1: track 11.7 -> 0.00 mm
- net SOL6_1: track 11.2 -> 0.00 mm
- added copper zone on layer 1, net 12V_GND
- removed copper zone on layer 1, net GND

Commit message: Add files via upload
Parts:
- removed D1, D2: HLMP6, display-hp:HLMP6
- removed TP1, TP2, TP3, TP4, TP5, TP6, TP7: TEST-POINT3, SparkFun-Connectors:PAD.03X.03
- added D3, D4: (no value), SparkFun-LED:LED-0805
- added J10, J11, J5, J6, J7, J8, J9: (no value), SparkFun-Connectors:1X01
- added J12, J13: 282837-3, X16_Backplane:TE_282837-3
- J3: value SAMTEC-HTST-110-04-X-D-RAJ -> HTST-110-04-L-D-RA; device X16_Backplane:SAMTEC-HTST-110-04-X-D-RA -> X16_Backplane:CONN_HTST-110-04/05-X-D-RA_SAI
- moved R1 104.5 mm to (-3.05, -15.5), flipped to the top
- moved R2 101.8 mm to (2.03, -9.40), flipped to the top
- moved C3 57.9 mm to (119.9, 39.1), flipped to the top
- moved C1 50.3 mm to (36.8, 38.9), flipped to the top
- moved J1 22.1 mm to (128.0, 106.7), flipped to the top
- moved J3 16.9 mm to (16.3, 99.3), flipped to the top
- moved J4 9.12 mm to (70.1, 70.6), flipped to the top
- moved C2 2.03 mm to (72.6, 39.1), flipped to the top
- moved J2 1.52 mm to (9.65, 55.0), flipped to the top
- moved U2 1.52 mm to (116.8, 93.0), flipped to the top
Connections:
- new net CLK: J3.9
- net 12V: now also D4.A, J12.1, J13.1, J5.1; no longer D1.A, TP1.1
- net 12V_GND: now also C1.2, C2.2, C3.2
- net 5V: now also D3.A, J3.20, J6.1; no longer D2.A, J3.1, TP2.1
- net CS: now also J11.1, J3.7; no longer J3.20, TP7.1
- net CTRL: now also J3.16; no longer J3.7
- net GND: now also J12.3, J13.3, J3.4, J7.1; no longer C1.2, C2.2, C3.2, J3.3, TP3.1
- net GPIO1: now also J3.1; no longer J3.2
- net GPIO2: now also J3.13; no longer J3.4
- net GPIO3: now also J3.14; no longer J3.6
- net GPIO4: now also J3.10; no longer J3.8
- net GPIO5: now also J3.8; no longer J3.9
- net GPIO6: now also J3.6; no longer J3.5
- net GPIO7: now also J3.5; no longer J3.10
- net GPIO8: now also J3.18; no longer J3.12
- net MISO: now also J3.12, J8.1; no longer J3.14, TP4.1
- net MOSI: now also J3.11, J9.1; no longer J3.16, TP5.1
- net N$2: now also D4.C; no longer D1.K
- net N$5: now also D3.C; no longer D2.K
- net PWMC0: now also J12.2
- net PWMC1: now also J13.2
- net SA0: now also J3.2; no longer J3.17
- net SA1: now also J3.15; no longer J3.19
- net SALERT: now also J3.3; no longer J3.13
- net SCL: now also J3.17; no longer J3.15
- net SCLK: now also J10.1; no longer J3.18, TP6.1
- net SDA: now also J3.19; no longer J3.11
Routing:
- net PWMC0: track 0.00 -> 71.3 mm
- net PWMC1: track 0.00 -> 69.0 mm
- net PWMC2: track 0.00 -> 66.2 mm
- net PWMC3: track 0.00 -> 63.4 mm
- net MISO: track 0.00 -> 57.6 mm, vias 0 -> 1
- net MOSI: track 0.00 -> 54.7 mm, vias 0 -> 1
- net GND: track 48.5 -> 0.00 mm
- net PWMB2: track 0.00 -> 48.2 mm, vias 0 -> 1
- net PWMB3: track 0.00 -> 47.5 mm, vias 0 -> 1
- net N$5: track 4.34 -> 0.00 mm
- net N$2: track 3.81 -> 0.00 mm
- net 12V: track 0.00 -> 2.16 mm
- net 5V: track 97.0 -> 98.0 mm
- added copper zone on layer 1, net 5V
- added copper zone on layer 1, net GND
- added copper zone on layer 16, net GND
