File: X16-Backplane1.brd (EAGLE design)
At the start: 139.7 x 110 mm, 24 parts, among them J1 CONN_PXC-8-RA-1778683, J12 282837-3, J13 282837-3, J2 CONN_ET60S-D04-3-08-D04-X-R1-S, J3 HTST-110-04-L-D-RA, J4 CLT-110-01-F-D, U2 TRANS_ULN2003AD

Commit message: Add files via upload
Parts:
- moved C2 14.5 mm to (87.1, 38.9)
- moved C3 11.7 mm to (131.6, 38.6)
- moved C1 4.57 mm to (41.4, 38.9)
- moved R2 3.64 mm to (0.51, -12.7)
- moved U2 0.25 mm to (116.6, 93.0)
Connections:
- removed net CLK: J3.9
- net SCLK: now also J3.9
Routing:
- net 12V: track 2.16 -> 163.6 mm, vias 0 -> 2
- net GPIO1: track 0.00 -> 133.3 mm, vias 0 -> 4
- net GPIO7: track 0.00 -> 128.1 mm, vias 0 -> 1
- net GPIO6: track 0.00 -> 127.4 mm, vias 0 -> 2
- net GPIO5: track 0.00 -> 121.3 mm, vias 0 -> 1
- net GPIO4: track 0.00 -> 114.8 mm, vias 0 -> 1
- net CTRL: track 0.00 -> 102.5 mm, vias 0 -> 1
- net GPIO2: track 0.00 -> 96.1 mm, vias 0 -> 2
- net PWMC1: track 69.0 -> 163.0 mm, vias 0 -> 3
- net GPIO3: track 0.00 -> 90.8 mm, vias 0 -> 2
- net 5V: track 98.0 -> 187.8 mm
- net PWMC0: track 71.3 -> 159.0 mm, vias 0 -> 1
- net SDA: track 0.00 -> 87.2 mm, vias 0 -> 2
- net SA1: track 0.00 -> 85.2 mm, vias 0 -> 1
- net SCL: track 0.00 -> 77.1 mm, vias 0 -> 1
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
Commit message: Add files via upload
Routing:
- net PWMA0: track 39.5 -> 38.0 mm
- net 5V: track 187.8 -> 187.1 mm
Changed lines of the file:
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@@
 <contactref element="U$1" pad="PWM0"/>
 <contactref element="J4" pad="13"/>
-<wire x1="73.104" y1="72.122" x2="60.39" y2="84.836" width="0.2032" layer="1"/>
-<wire x1="60.39" y1="84.836" x2="41.402" y2="84.836" width="0.2032" layer="1"/>
-<wire x1="41.402" y1="84.836" x2="41.402" y2="87.376" width="0.2032" layer="1"/>
+<wire x1="59.882" y1="85.344" x2="43.434" y2="85.344" width="0.2032" layer="1"/>
+<wire x1="43.434" y1="85.344" x2="41.402" y2="87.376" width="0.2032" layer="1"/>
+<wire x1="73.104" y1="72.122" x2="59.882" y2="85.344" width="0.2032" layer="1"/>
 </signal>
 <signal name="PWMA1">
@@
 <contactref element="U$2" pad="PWM2"/>
 <contactref element="J4" pad="10"/>
-<wire x1="70.104" y1="67.056" x2="82.55" y2="67.056" width="0.2032" layer="16"/>
-<wire x1="82.55" y1="67.056" x2="83.058" y2="67.564" width="0.2032" layer="16"/>
-<wire x1="83.058" y1="67.564" x2="83.058" y2="91.44" width="0.2032" layer="16"/>
-<wire x1="83.058" y1="91.44" x2="84.074" y2="92.456" width="0.2032" layer="16"/>
+<wire x1="70.104" y1="67.056" x2="82.296" y2="67.056" width="0.2032" layer="16"/>
+<wire x1="82.296" y1="67.056" x2="83.312" y2="68.072" width="0.2032" layer="16"/>
+<wire x1="83.312" y1="68.072" x2="83.312" y2="91.694" width="0.2032" layer="16"/>
+<wire x1="83.312" y1="91.694" x2="84.074" y2="92.456" width="0.2032" layer="16"/>
 <wire x1="84.074" y1="92.456" x2="87.122" y2="92.456" width="0.2032" layer="16"/>
 <wire x1="70.104" y1="67.056" x2="69.104" y2="68.056" width="0.2032" layer="16"/>
@@
 <contactref element="J4" pad="12"/>
 <wire x1="71.104" y1="69.102" x2="71.12" y2="69.086" width="0.2032" layer="1"/>
-<wire x1="81.788" y1="93.726" x2="81.788" y2="68.072" width="0.2032" layer="16"/>
-<wire x1="81.788" y1="93.726" x2="83.058" y2="94.996" width="0.2032" layer="16"/>
+<wire x1="82.296" y1="94.234" x2="82.296" y2="68.58" width="0.2032" layer="16"/>
+<wire x1="82.296" y1="94.234" x2="83.058" y2="94.996" width="0.2032" layer="16"/>
 <wire x1="83.058" y1="94.996" x2="87.122" y2="94.996" width="0.2032" layer="16"/>
 <wire x1="71.104" y1="68.596" x2="71.104" y2="69.102" width="0.2032" layer="16"/>
 <wire x1="72.136" y1="67.564" x2="71.104" y2="68.596" width="0.2032" layer="16"/>
-<wire x1="81.788" y1="68.072" x2="81.28" y2="67.564" width="0.2032" layer="16"/>
+<wire x1="82.296" y1="68.58" x2="81.28" y2="67.564" width="0.2032" layer="16"/>
 <wire x1="81.28" y1="67.564" x2="72.136" y2="67.564" width="0.2032" layer="16"/>
 </signal>
@@
 <wire x1="80.264" y1="94.996" x2="80.264" y2="75.438" width="0.2032" layer="1"/>
 <wire x1="80.264" y1="75.438" x2="81.026" y2="74.676" width="0.2032" layer="1"/>
-<wire x1="81.026" y1="74.676" x2="106.426" y2="74.676" width="0.2032" layer="1"/>
-<via x="106.426" y="74.676" extent="1-16" drill="0.35"/>
-<wire x1="122.682" y1="74.676" x2="106.426" y2="74.676" width="0.2032" layer="16"/>
+<wire x1="81.026" y1="74.676" x2="106.68" y2="74.676" width="0.2032" layer="1"/>
+<via x="106.68" y="74.676" extent="1-16" drill="0.35"/>
+<wire x1="106.68" y1="74.676" x2="122.682" y2="74.676" width="0.2032" layer="16"/>
 <wire x1="122.682" y1="74.676" x2="131.572" y2="83.566" width="0.2032" layer="16"/>
 <wire x1="131.572" y1="83.566" x2="131.572" y2="87.376" width="0.2032" layer="16"/>
@@
 <wire x1="56.6920875" y1="101.854" x2="58.6450875" y2="99.901" width="0.3048" layer="16"/>
 <wire x1="91.615" y1="99.901" x2="93.218" y2="98.298" width="0.3048" layer="16"/>
-<wire x1="93.218" y1="98.298" x2="93.218" y2="65.278" width="0.3048" layer="16"/>
-<wire x1="93.218" y1="65.278" x2="92.202" y2="64.262" width="0.3048" layer="16"/>
-<wire x1="92.202" y1="64.262" x2="60.452" y2="64.262" width="0.3048" layer="16"/>
+<wire x1="93.218" y1="98.298" x2="93.218" y2="66.548" width="0.3048" layer="16"/>
+<wire x1="93.218" y1="66.548" x2="90.932" y2="64.262" width="0.3048" layer="16"/>
+<wire x1="90.932" y1="64.262" x2="60.452" y2="64.262" width="0.3048" layer="16"/>
 <wire x1="60.452" y1="64.262" x2="57.658" y2="67.056" width="0.3048" layer="16"/>
 <wire x1="57.658" y1="67.056" x2="57.658" y2="71.374" width="0.3048" layer="16"/>
@@
 <wire x1="38.1" y1="84.836" x2="40.64" y2="84.836" width="0.2032" layer="1"/>
 <via x="40.64" y="84.836" extent="1-16" drill="0.35"/>
-<wire x1="40.64" y1="84.836" x2="81.28" y2="84.836" width="0.2032" layer="16"/>
+<wire x1="81.28" y1="84.836" x2="40.64" y2="84.836" width="0.2032" layer="16"/>
 <via x="81.28" y="84.836" extent="1-16" drill="0.35"/>
 <wire x1="81.28" y1="84.836" x2="109.728" y2="84.836" width="0.2032" layer="1"/>
@@
 <contactref element="J3" pad="5"/>
 <wire x1="119.761" y1="90.489" x2="119.761" y2="87.249" width="0.2032" layer="1"/>
-<wire x1="119.761" y1="87.249" x2="108.0742" y2="75.5622" width="0.2032" layer="1"/>
+<wire x1="119.761" y1="87.249" x2="108.3112" y2="75.7992" width="0.2032" layer="1"/>
 <via x="81.28" y="75.5452" extent="1-16" drill="0.35"/>
-<wire x1="106.16413125" y1="75.5622" x2="106.14713125" y2="75.5452" width="0.2032" layer="1"/>
-<wire x1="106.14713125" y1="75.5452" x2="81.28" y2="75.5452" width="0.2032" layer="1"/>
-<wire x1="108.0742" y1="75.5622" x2="106.16413125" y2="75.5622" width="0.2032" layer="1"/>
+<wire x1="108.3112" y1="75.7992" x2="81.534" y2="75.7992" width="0.2032" layer="1"/>
+<wire x1="81.534" y1="75.7992" x2="81.28" y2="75.5452" width="0.2032" layer="1"/>
 <wire x1="81.28" y1="75.5452" x2="25.0388" y2="75.5452" width="0.2032" layer="16"/>
 <wire x1="25.0388" y1="75.5452" x2="21.336" y2="79.248" width="0.2032" layer="16"/>

Commit message: Add files via upload
Parts:
- moved D3 7.89 mm to (-1.78, -8.38)
Changed lines of the file:
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@@
 <attribute name="VALUE" x="68.103290625" y="111.11381875" size="1.27085" layer="27" rot="R180"/>
 </element>
-<element name="D3" library="SparkFun-LED" library_urn="urn:adsk.eagle:library:529" package="LED-0805" package3d_urn="urn:adsk.eagle:package:41389318/1" value="" x="-8.382" y="-4.064" smashed="yes">
-<attribute name="NAME" x="-8.382" y="-3.064" size="0.6096" layer="25" font="vector" ratio="20" align="bottom-center"/>
-<attribute name="VALUE" x="-8.382" y="-5.064" size="0.6096" layer="27" font="vector" ratio="20" align="top-center"/>
+<element name="D3" library="SparkFun-LED" library_urn="urn:adsk.eagle:library:529" package="LED-0805" package3d_urn="urn:adsk.eagle:package:41389318/1" value="" x="-1.778" y="-8.382" smashed="yes">
+<attribute name="NAME" x="-1.778" y="-7.382" size="0.6096" layer="25" font="vector" ratio="20" align="bottom-center"/>
+<attribute name="VALUE" x="-1.778" y="-9.382" size="0.6096" layer="27" font="vector" ratio="20" align="top-center"/>
 </element>
 <element name="D4" library="SparkFun-LED" library_urn="urn:adsk.eagle:library:529" package="LED-0805" package3d_urn="urn:adsk.eagle:package:41389318/1" value="" x="-8.382" y="-7.112" smashed="yes">
@@
 <wire x1="58.406" y1="72.122" x2="61.104" y2="72.122" width="0.3048" layer="16"/>
 <wire x1="39.116" y1="101.854" x2="78.232" y2="136.906" width="0" layer="19" extent="1-1"/>
-<wire x1="-9.432" y1="-4.064" x2="4.652" y2="79.879890625" width="0" layer="19" extent="1-1"/>
+<wire x1="-2.828" y1="-8.382" x2="4.652" y2="79.879890625" width="0" layer="19" extent="1-1"/>
 </signal>
 <signal name="CTRL">
@@
 <contactref element="J9" pad="1"/>
 <contactref element="J3" pad="11"/>
-<wire x1="67.104" y1="72.122" x2="61.502" y2="77.724" width="0.2032" layer="1"/>
-<wire x1="30.988" y1="77.724" x2="28.956" y2="79.756" width="0.2032" layer="1"/>
+<wire x1="67.104" y1="72.122" x2="62.01" y2="77.216" width="0.2032" layer="1"/>
+<wire x1="31.496" y1="77.216" x2="28.956" y2="79.756" width="0.2032" layer="1"/>
 <wire x1="28.956" y1="79.756" x2="28.956" y2="99.314" width="0.2032" layer="1"/>
-<wire x1="61.502" y1="77.724" x2="30.988" y2="77.724" width="0.2032" layer="1"/>
+<wire x1="62.01" y1="77.216" x2="31.496" y2="77.216" width="0.2032" layer="1"/>
 <wire x1="67.104" y1="72.122" x2="89.662" y2="136.906" width="0" layer="19" extent="1-1"/>
 </signal>
@@
 <contactref element="R2" pad="2"/>
 <contactref element="D3" pad="C"/>
-<wire x1="1.358" y1="-12.7" x2="-7.332" y2="-4.064" width="0" layer="19" extent="1-1"/>
+<wire x1="-0.728" y1="-8.382" x2="1.358" y2="-12.7" width="0" layer="19" extent="1-1"/>
 </signal>
 <signal name="GPIO6">
@@
 <contactref element="U2" pad="5"/>
 <contactref element="J3" pad="8"/>
-<wire x1="81.026" y1="79.248" x2="26.162" y2="79.248" width="0.2032" layer="16"/>
-<wire x1="81.026" y1="79.248" x2="81.28" y2="78.994" width="0.2032" layer="16"/>
+<wire x1="80.518" y1="79.756" x2="25.654" y2="79.756" width="0.2032" layer="16"/>
+<wire x1="80.518" y1="79.756" x2="81.28" y2="78.994" width="0.2032" layer="16"/>
 <via x="81.28" y="78.994" extent="1-16" drill="0.35"/>
 <wire x1="81.28" y1="78.994" x2="83.058" y2="80.772" width="0.2032" layer="1"/>
@@
 <wire x1="23.876" y1="100.75084375" x2="23.876" y2="101.854" width="0.2032" layer="16"/>
 <wire x1="22.86" y1="99.73484375" x2="23.876" y2="100.75084375" width="0.2032" layer="16"/>
-<wire x1="26.162" y1="79.248" x2="22.86" y2="82.55" width="0.2032" layer="16"/>
+<wire x1="25.654" y1="79.756" x2="22.86" y2="82.55" width="0.2032" layer="16"/>
 <wire x1="22.86" y1="82.55" x2="22.86" y2="99.73484375" width="0.2032" layer="16"/>
 </signal>
@@
 <wire x1="108.3112" y1="75.7992" x2="81.534" y2="75.7992" width="0.2032" layer="1"/>
 <wire x1="81.534" y1="75.7992" x2="81.28" y2="75.5452" width="0.2032" layer="1"/>
-<wire x1="81.28" y1="75.5452" x2="25.0388" y2="75.5452" width="0.2032" layer="16"/>
-<wire x1="25.0388" y1="75.5452" x2="21.336" y2="79.248" width="0.2032" layer="16"/>
+<wire x1="81.28" y1="75.5452" x2="80.518" y2="76.3072" width="0.2032" layer="16"/>
+<wire x1="80.518" y1="76.3072" x2="24.2768" y2="76.3072" width="0.2032" layer="16"/>
+<wire x1="24.2768" y1="76.3072" x2="21.336" y2="79.248" width="0.2032" layer="16"/>
 <wire x1="21.336" y1="79.248" x2="21.336" y2="99.314" width="0.2032" layer="16"/>
 </signal>

Commit message: Add files via upload
Parts:
- moved D3 97.9 mm to (54.4, 71.9), turned to 180 degrees
- moved R2 97.8 mm to (54.1, 69.1), turned to 180 degrees
- moved R1 61.3 mm to (29.2, 36.6)
- moved D4 56.4 mm to (31.1, 33.1), turned to 180 degrees
Routing:
- net 12V: track 163.6 -> 176.5 mm
- net 5V: track 187.1 -> 194.3 mm
- net N$2: track 0.00 -> 3.43 mm
- net N$5: track 0.00 -> 2.82 mm

Commit message: Add files via upload
Parts:
- removed J5, J6, J7: (no value), SparkFun-Connectors:1X01
- added H1, H2, H3, H4: 6-32-HOLE, X16-ExtraComponents:6-32-HOLE
- added TP1, TP2, TP3, TP4: TESTPOINT_5.04MM, X16_Backplane:TESTPOINT_5.04MM
- U$1, U$2, U$3: value CONN_BACKPLANE_ESC_ADAPTER -> CONN_BACKPLANE_ESC_ADAPTER_NEW
- moved J12 99.4 mm to (78.7, 5.84)
- moved J13 99.3 mm to (57.7, 6.10)
- moved J8 36.1 mm to (67.8, 105.7)
- moved J9 35.5 mm to (72.9, 105.7)
- moved J10 35.1 mm to (78.0, 105.4)
- moved J11 35.0 mm to (82.5, 105.2)
- moved R1 25.2 mm to (54.4, 35.3)
- moved D4 23.1 mm to (54.2, 32.1), turned to 0 degrees
- moved U2 7.73 mm to (117.9, 85.3)
- moved J1 7.62 mm to (128.0, 99.1)
- moved D3 4.99 mm to (55.6, 76.7)
- moved R2 4.71 mm to (53.7, 73.8), turned to 0 degrees
- moved J4 4.57 mm to (70.1, 75.2)
Connections:
- net 12V: now also TP1.TP; no longer J5.1
- net 12V_GND: now also J12.3, J13.3, R1.1, TP2.TP
- net 12V_L: now also J2.08, J2.16, J2.24
- net 5V: now also TP3.TP; no longer J6.1
- net GND: now also TP4.TP, U$1.NC@1, U$1.NC@2, U$1.NC@3, U$1.NC@4, U$1.NC@5, U$1.NC@6, U$2.NC@1, U$2.NC@2, U$2.NC@3, U$2.NC@4, U$2.NC@5, U$2.NC@6, U$3.NC@1, U$3.NC@2, U$3.NC@3, U$3.NC@4, U$3.NC@5, U$3.NC@6; no longer J12.3, J13.3, J7.1, R1.1
Routing:
- net 12V_L: track 7.53 -> 185.4 mm
- net 12V_GND: track 24.5 -> 180.4 mm
- net PWMC1: track 162.6 -> 266.5 mm, vias 3 -> 1
- net GND: track 0.00 -> 97.0 mm, vias 0 -> 2
- net PWMC0: track 159.0 -> 255.6 mm
- net 12V: track 176.5 -> 96.4 mm, vias 2 -> 0
- net 5V: track 194.3 -> 134.1 mm, vias 0 -> 4
- net SCLK: track 63.5 -> 115.1 mm, vias 1 -> 3
- net MOSI: track 60.9 -> 100.2 mm, vias 0 -> 3
- net CS: track 68.2 -> 97.5 mm
- net SA1: track 85.2 -> 62.1 mm, vias 1 -> 2
- net GPIO1: track 133.3 -> 112.9 mm, vias 4 -> 1
- net SALERT: track 68.5 -> 54.8 mm
- net GPIO7: track 128.1 -> 115.0 mm, vias 1 -> 0
- net GPIO6: track 127.4 -> 114.5 mm, vias 2 -> 0
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
Commit message: Add files via upload
Routing:
- net SDA: track 95.0 -> 93.4 mm
- net 12V: track 96.4 -> 94.8 mm
- net SA1: track 62.1 -> 61.3 mm

Commit message: Add files via upload
Parts:
- moved J8 0.25 mm to (67.8, 105.4)
- moved J9 0.25 mm to (72.9, 105.4)
- moved J11 0.25 mm to (82.5, 105.4)
Other:
- board text added: "12V"
- board text added: "12V_GND"
- board text added: "5V"
- board text added: "CS"
- board text added: "GND"
- board text added: "MISO"
- board text added: "MOSI"
- board text added: "SCLK"
Changed lines of the file:
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@@
 <vertex x="23.368" y="35.052"/>
 </polygon>
+<text x="66.929" y="106.934" size="0.508" layer="25">MISO</text>
+<text x="73.406" y="106.934" size="0.508" layer="25">MOSI</text>
+<text x="80.264" y="107.442" size="0.508" layer="25" rot="R180">SCLK</text>
+<text x="83.058" y="107.442" size="0.508" layer="25" rot="R180">CS</text>
+<text x="93.599" y="101.092" size="1.27" layer="25" rot="R180">5V</text>
+<text x="105.156" y="101.219" size="1.27" layer="25" rot="R180">GND</text>
+<text x="139.192" y="79.502" size="1.27" layer="25" rot="R180">12V_GND</text>
+<text x="24.892" y="7.62" size="1.27" layer="25" rot="R180">12V</text>
 </plain>
 <attributes>
@@
 <attribute name="VALUE" x="80.009" y="78.994" size="1.27" layer="27" rot="R180"/>
 </element>
-<element name="J8" library="SparkFun-Connectors" library_urn="urn:adsk.eagle:library:513" package="1X01" package3d_urn="urn:adsk.eagle:package:38028/2" value="" x="67.818" y="105.664" smashed="yes" rot="R90">
-<attribute name="NAME" x="66.421" y="104.394" size="0.6096" layer="25" font="vector" ratio="20" rot="R90"/>
-<attribute name="VALUE" x="69.342" y="104.394" size="0.6096" layer="27" font="vector" ratio="20" rot="R90" align="top-left"/>
-</element>
-<element name="J9" library="SparkFun-Connectors" library_urn="urn:adsk.eagle:library:513" package="1X01" package3d_urn="urn:adsk.eagle:package:38028/2" value="" x="72.898" y="105.664" smashed="yes" rot="R90">
-<attribute name="NAME" x="71.501" y="104.394" size="0.6096" layer="25" font="vector" ratio="20" rot="R90"/>
-<attribute name="VALUE" x="74.422" y="104.394" size="0.6096" layer="27" font="vector" ratio="20" rot="R90" align="top-left"/>
+<element name="J8" library="SparkFun-Connectors" library_urn="urn:adsk.eagle:library:513" package="1X01" package3d_urn="urn:adsk.eagle:package:38028/2" value="" x="67.818" y="105.41" smashed="yes" rot="R90">
+<attribute name="NAME" x="66.421" y="104.14" size="0.6096" layer="25" font="vector" ratio="20" rot="R90"/>
+<attribute name="VALUE" x="69.342" y="104.14" size="0.6096" layer="27" font="vector" ratio="20" rot="R90" align="top-left"/>
+</element>
+<element name="J9" library="SparkFun-Connectors" library_urn="urn:adsk.eagle:library:513" package="1X01" package3d_urn="urn:adsk.eagle:package:38028/2" value="" x="72.898" y="105.41" smashed="yes" rot="R90">
+<attribute name="NAME" x="71.501" y="104.14" size="0.6096" layer="25" font="vector" ratio="20" rot="R90"/>
+<attribute name="VALUE" x="74.422" y="104.14" size="0.6096" layer="27" font="vector" ratio="20" rot="R90" align="top-left"/>
 </element>
 <element name="J10" library="SparkFun-Connectors" library_urn="urn:adsk.eagle:library:513" package="1X01" package3d_urn="urn:adsk.eagle:package:38028/2" value="" x="77.978" y="105.41" smashed="yes" rot="R90">
@@
 <attribute name="VALUE" x="79.502" y="104.14" size="0.6096" layer="27" font="vector" ratio="20" rot="R90" align="top-left"/>
 </element>
-<element name="J11" library="SparkFun-Connectors" library_urn="urn:adsk.eagle:library:513" package="1X01" package3d_urn="urn:adsk.eagle:package:38028/2" value="" x="82.55" y="105.156" smashed="yes" rot="R90">
-<attribute name="NAME" x="81.153" y="103.886" size="0.6096" layer="25" font="vector" ratio="20" rot="R90"/>
-<attribute name="VALUE" x="84.074" y="103.886" size="0.6096" layer="27" font="vector" ratio="20" rot="R90" align="top-left"/>
+<element name="J11" library="SparkFun-Connectors" library_urn="urn:adsk.eagle:library:513" package="1X01" package3d_urn="urn:adsk.eagle:package:38028/2" value="" x="82.55" y="105.41" smashed="yes" rot="R90">
+<attribute name="NAME" x="81.153" y="104.14" size="0.6096" layer="25" font="vector" ratio="20" rot="R90"/>
+<attribute name="VALUE" x="84.074" y="104.14" size="0.6096" layer="27" font="vector" ratio="20" rot="R90" align="top-left"/>
 </element>
 <element name="J12" library="X16_Backplane" package="TE_282837-3" value="282837-3" x="78.74" y="5.842" smashed="yes" rot="R180">
@@
 <wire x1="52.578" y1="4.318" x2="52.578" y2="6.096" width="0.762" layer="1"/>
 <wire x1="53.506" y1="43.014" x2="53.506" y2="35.306" width="1.524" layer="1"/>
-<wire x1="41.402" y1="45.212" x2="51.308" y2="45.212" width="1.524" layer="1"/>
+<wire x1="51.308" y1="45.212" x2="41.402" y2="45.212" width="1.524" layer="1"/>
 <wire x1="51.308" y1="45.212" x2="53.506" y2="43.014" width="1.524" layer="1"/>
 <contactref element="TP2" pad="TP"/>
@@
 <wire x1="87.122" y1="55.626" x2="87.122" y2="42.4688" width="1.524" layer="1"/>
 <wire x1="131.572" y1="55.626" x2="131.572" y2="42.2148" width="1.524" layer="1"/>
-<wire x1="41.402" y1="55.626" x2="41.402" y2="42.4688" width="1.524" layer="1"/>
-<wire x1="41.402" y1="42.4688" x2="41.402" y2="45.212" width="0" layer="19" extent="1-1"/>
+<wire x1="41.402" y1="42.4688" x2="41.402" y2="45.212" width="1.524" layer="1"/>
+<wire x1="41.402" y1="45.212" x2="41.402" y2="55.626" width="1.524" layer="1"/>
 </signal>
 <signal name="PWMB0">
@@
 <via x="60.706" y="103.3808" extent="1-16" drill="0.35"/>
 <wire x1="60.706" y1="103.3808" x2="60.706" y2="102.362" width="0.2032" layer="1"/>
-<wire x1="67.818" y1="105.664" x2="65.786" y2="105.664" width="0.2032" layer="16"/>
-<wire x1="65.786" y1="105.664" x2="64.262" y2="107.188" width="0.2032" layer="16"/>
+<wire x1="67.818" y1="105.41" x2="66.04" y2="105.41" width="0.2032" layer="16"/>
+<wire x1="66.04" y1="105.41" x2="64.262" y2="107.188" width="0.2032" layer="16"/>
 <wire x1="64.262" y1="107.188" x2="60.96" y2="107.188" width="0.2032" layer="16"/>
 <wire x1="60.96" y1="107.188" x2="60.706" y2="106.934" width="0.2032" layer="16"/>
@@
 <wire x1="27.686" y1="101.6" x2="28.956" y2="100.33" width="0.2032" layer="1"/>
 <wire x1="28.956" y1="100.33" x2="28.956" y2="99.314" width="0.2032" layer="1"/>
-<wire x1="72.898" y1="104.394" x2="72.898" y2="105.664" width="0.2032" layer="16"/>
+<wire x1="72.898" y1="104.394" x2="72.898" y2="105.41" width="0.2032" layer="16"/>
 <wire x1="72.323965625" y1="103.819965625" x2="62.417965625" y2="103.819965625" width="0.2032" layer="16"/>
 <via x="62.417965625" y="103.819965625" extent="1-16" drill="0.35"/>
@@
 <wire x1="61.401965625" y1="103.819965625" x2="61.341" y2="103.759" width="0.2032" layer="1"/>
 <wire x1="72.898" y1="104.394" x2="72.323965625" y2="103.819965625" width="0.2032" layer="16"/>
-<wire x1="72.898" y1="105.664" x2="72.898" y2="107.188" width="0.2032" layer="16"/>
+<wire x1="72.898" y1="105.41" x2="72.898" y2="107.188" width="0.2032" layer="16"/>
 <wire x1="72.898" y1="107.188" x2="72.39" y2="107.696" width="0.2032" layer="16"/>
 <wire x1="72.39" y1="107.696" x2="59.436" y2="107.696" width="0.2032" layer="16"/>
@@
 <wire x1="22.606" y1="101.6" x2="23.876" y2="100.33" width="0.2032" layer="1"/>
 <wire x1="23.876" y1="100.33" x2="23.876" y2="99.314" width="0.2032" layer="1"/>
-<wire x1="82.55" y1="105.156" x2="82.55" y2="103.886" width="0.2032" layer="1"/>
+<wire x1="82.55" y1="105.41" x2="82.55" y2="103.886" width="0.2032" layer="1"/>
 <wire x1="82.55" y1="103.886" x2="80.772" y2="102.108" width="0.2032" layer="1"/>
 <wire x1="80.772" y1="102.108" x2="67.056" y2="102.108" width="0.2032" layer="1"/>

Commit message: Add files via upload
Parts:
- moved C3 10.2 mm to (121.4, 38.9)
- moved U2 8.89 mm to (109.0, 85.1)
- moved J1 8.89 mm to (119.1, 99.1)
- moved TP2 8.70 mm to (125.7, 73.4)
- moved H2 8.38 mm to (126.5, 105.4)
- moved H4 8.38 mm to (126.5, 4.57)
- moved U$3 5.84 mm to (89.4, 106.7)
- moved C2 3.57 mm to (83.6, 38.6)
- moved U$2 3.56 mm to (47.2, 106.7)
Routing:
- net PWMC0: track 255.6 -> 234.9 mm
- net 12V_L: track 185.4 -> 175.4 mm
- net GPIO4: track 105.3 -> 96.4 mm
- net GPIO1: track 112.9 -> 104.1 mm
- net GPIO2: track 95.0 -> 86.2 mm
- net GPIO3: track 98.6 -> 89.8 mm
- net GPIO5: track 109.7 -> 101.2 mm
- net GPIO6: track 114.5 -> 106.4 mm
- net GPIO7: track 115.0 -> 107.4 mm
- net PWMC3: track 67.4 -> 62.2 mm
- net PWMC1: track 266.0 -> 261.1 mm
- net PWMC2: track 69.3 -> 64.9 mm
- net PWMB0: track 34.1 -> 30.5 mm
- net PWMB1: track 36.7 -> 33.2 mm
- net PWMB2: track 43.9 -> 40.8 mm
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Other:
- board size 139.7 x 110 mm -> 131.3 x 110.3 mm
