File: X16-Backplane1.sch (EAGLE design)
At the start: 15 parts, among them J1 CONN_PXC-8-RA-1778683, J2 CONN_ET60S-D04-3-08-D04-X-R1-S, J3 SAMTEC-HTST-110-04-X-D-RAJ, J4 SAMTEC-HTST-110-04-X-D-RAJ, U1 TRANS_ULN2003AD

Commit message: Add files via upload
Parts:
- removed J4: SAMTEC-HTST-110-04-X-D-RAJ, X16_Backplane:SAMTEC-HTST-110-04-X-D-RAJ
- removed U1: TRANS_ULN2003AD, X16_Backplane:TRANS_ULN2003AD
- added J5: SAMTEC-HTST-110-04-X-D-RAJ, X16_Backplane:SAMTEC-HTST-110-04-X-D-RAJ
- added TP1, TP2, TP3, TP4, TP5, TP6, TP7: TEST-POINT3, SparkFun-Connectors:TEST-POINT3
- added U2: TRANS_ULN2003AD, X16_Backplane:TRANS_ULN2003AD
Connections:
- net 12V: now also TP1.1
- net 12V_L: now also U2.COM; no longer U1.COM
- net 5V: now also J5.1, J5.3, TP2.1; no longer J3.3, J4.1
- net CS: now also J3.20, J5.11, TP7.1; no longer J3.11, J4.20
- net CTRL: now also J3.7; no longer J4.7
- net DGND: now also J3.9; no longer J4.9
- net GND: now also J3.3, J5.2, J5.4, TP3.1, U2.GND; no longer J3.2, J3.4, J4.3, U1.GND
- net GPIO1: now also J3.2, U2.IN1; no longer J4.2, U1.IN1
- net GPIO2: now also J3.4, U2.IN2; no longer J4.4, U1.IN2
- net GPIO3: now also J3.6, U2.IN3; no longer J4.6, U1.IN3
- net GPIO4: now also J3.8, U2.IN4; no longer J4.8, U1.IN4
- net MISO: now also J3.14, J5.5, TP4.1; no longer J3.5, J4.14
- net MOSI: now also J3.16, J5.7, TP5.1; no longer J3.7, J4.16
- net PWMA0: now also J5.13; no longer J3.13
- net PWMA1: now also J5.15; no longer J3.15
- net PWMA2: now also J5.17; no longer J3.17
- net PWMA3: now also J5.19; no longer J3.19
- net PWMB0: now also J5.6; no longer J3.6
- net PWMB1: now also J5.8; no longer J3.8
- net PWMB2: now also J5.10; no longer J3.10
- net PWMB3: now also J5.12; no longer J3.12
- net PWMC0: now also J5.14; no longer J3.14
- net PWMC1: now also J5.16; no longer J3.16
- net PWMC2: now also J5.18; no longer J3.18
- net PWMC3: now also J5.20; no longer J3.20
- net SA0: now also J3.17; no longer J4.17
- net SA1: now also J3.19; no longer J4.19
- net SALERT: now also J3.13; no longer J4.13
- net SCL: now also J3.15; no longer J4.15
- net SCLK: now also J3.18, J5.9, TP6.1; no longer J3.9, J4.18
- net SDA: now also J3.11; no longer J4.11
- net SOL1_1: now also U2.OUT1; no longer U1.OUT1
- net SOL2_1: now also U2.OUT2; no longer U1.OUT2
- net SOL3_1: now also U2.OUT3; no longer U1.OUT3
- net SOL4_1: now also U2.OUT4; no longer U1.OUT4
Other:
- note added: "SOLENOID CONNECTOR"
- note added: "SOLENOID TRANSISTOR"
- moved on the sheet: D1, D2, J1, J2, R1, R2

Commit message: Add files via upload
Parts:
- removed J5: SAMTEC-HTST-110-04-X-D-RAJ, X16_Backplane:SAMTEC-HTST-110-04-X-D-RAJ
- added J4: CLT-110-01-F-D, X16_Backplane:CLT-110-01-F-D
Connections:
- net 5V: now also J4.01, J4.03; no longer J5.1, J5.3
- net CS: now also J4.11; no longer J5.11
- net GND: now also J4.02, J4.04; no longer J5.2, J5.4
- net MISO: now also J4.05; no longer J5.5
- net MOSI: now also J4.07; no longer J5.7
- net PWMA0: now also J4.13; no longer J5.13
- net PWMA1: now also J4.15; no longer J5.15
- net PWMA2: now also J4.17; no longer J5.17
- net PWMA3: now also J4.19; no longer J5.19
- net PWMB0: now also J4.06; no longer J5.6
- net PWMB1: now also J4.08; no longer J5.8
- net PWMB2: now also J4.10; no longer J5.10
- net PWMB3: now also J4.12; no longer J5.12
- net PWMC0: now also J4.14; no longer J5.14
- net PWMC1: now also J4.16; no longer J5.16
- net PWMC2: now also J4.18; no longer J5.18
- net PWMC3: now also J4.20; no longer J5.20
- net SCLK: now also J4.09; no longer J5.9

Commit message: Add files via upload
Connections:
- net 12V: now also C1.1, C2.1, C3.1; no longer C1.2, C2.2, C3.2
- net 12V_GND: no longer C1.1, C2.1, C3.1
- net GND: now also C1.2, C2.2, C3.2; no longer J1.7, J1.8, U2.GND
Other:
- note added: "+"
- moved on the sheet: C1, C2, C3
Changed lines of the file:
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@@
 <net name="GND" class="0">
-<segment>
-<pinref part="J1" gate="G$1" pin="7"/>
-<wire x1="50.8" y1="76.2" x2="58.42" y2="76.2" width="0.1524" layer="91"/>
-<wire x1="58.42" y1="76.2" x2="58.42" y2="73.66" width="0.1524" layer="91"/>
-<pinref part="J1" gate="G$1" pin="8"/>
-<wire x1="58.42" y1="73.66" x2="58.42" y2="66.04" width="0.1524" layer="91"/>
-<wire x1="50.8" y1="73.66" x2="58.42" y2="73.66" width="0.1524" layer="91"/>
-<junction x="58.42" y="73.66"/>
-<label x="58.42" y="66.04" size="1.778" layer="95"/>
-</segment>
 <segment>
 <pinref part="J2" gate="G$1" pin="P06"/>
@@
 </segment>
 <segment>
-<pinref part="U2" gate="G$1" pin="GND"/>
-<wire x1="109.22" y1="38.1" x2="109.22" y2="30.48" width="0.1524" layer="91"/>
-<label x="109.22" y="30.48" size="1.778" layer="95"/>
-</segment>
-<segment>
 <pinref part="J3" gate="A" pin="3"/>
 <wire x1="195.58" y1="88.9" x2="187.96" y2="88.9" width="0.1524" layer="91"/>
@@
 <text x="40.64" y="226.06" size="1.778" layer="91">12V LED CHECK</text>
 <text x="88.9" y="226.06" size="1.778" layer="91">5V LED CHECK</text>
-<text x="63.5" y="139.7" size="1.778" layer="91">12V CAPACITORS</text>
+<text x="66.04" y="160.02" size="1.778" layer="91">12V CAPACITORS</text>
+<text x="50.8" y="124.46" size="1.778" layer="91">+</text>
+<text x="73.66" y="124.46" size="1.778" layer="91">+</text>
+<text x="101.6" y="124.46" size="1.778" layer="91">+</text>
 </plain>
 <instances>
@@
 <attribute name="PROD_ID" x="90.17" y="198.12" size="1.778" layer="96" rot="MR90"/>
 </instance>
-<instance part="C1" gate="A" x="71.12" y="129.54" smashed="yes">
-<attribute name="VALUE" x="65.9638" y="124.0028" size="3.4798" layer="96" ratio="10" rot="SR0"/>
-<attribute name="NAME" x="67.0306" y="131.6228" size="3.4798" layer="95" ratio="10" rot="SR0"/>
-<attribute name="C1" x="78.74" y="132.08" size="1.778" layer="96"/>
-</instance>
-<instance part="C2" gate="A" x="71.12" y="106.68" smashed="yes">
-<attribute name="VALUE" x="65.9638" y="101.1428" size="3.4798" layer="96" ratio="10" rot="SR0"/>
-<attribute name="NAME" x="67.0306" y="108.7628" size="3.4798" layer="95" ratio="10" rot="SR0"/>
-<attribute name="C2" x="78.74" y="109.22" size="1.778" layer="96"/>
-</instance>
-<instance part="C3" gate="A" x="71.12" y="83.82" smashed="yes">
-<attribute name="VALUE" x="65.9638" y="78.2828" size="3.4798" layer="96" ratio="10" rot="SR0"/>
-<attribute name="NAME" x="67.0306" y="85.9028" size="3.4798" layer="95" ratio="10" rot="SR0"/>
-<attribute name="C3" x="78.74" y="86.36" size="1.778" layer="96"/>
+<instance part="C1" gate="A" x="53.34" y="127" smashed="yes" rot="R270">
+<attribute name="VALUE" x="30.0228" y="111.8362" size="3.4798" layer="96" ratio="10" rot="SR0"/>
+<attribute name="NAME" x="57.9628" y="123.4694" size="3.4798" layer="95" ratio="10" rot="SR0"/>
+<attribute name="C1" x="55.88" y="119.38" size="1.778" layer="96"/>
+</instance>
+<instance part="C2" gate="A" x="76.2" y="127" smashed="yes" rot="R270">
+<attribute name="VALUE" x="75.7428" y="111.8362" size="3.4798" layer="96" ratio="10" rot="SR0"/>
+<attribute name="NAME" x="80.8228" y="123.4694" size="3.4798" layer="95" ratio="10" rot="SR0"/>
+<attribute name="C2" x="78.74" y="119.38" size="1.778" layer="96"/>
+</instance>
+<instance part="C3" gate="A" x="104.14" y="127" smashed="yes" rot="R270">
+<attribute name="VALUE" x="116.3828" y="119.4562" size="3.4798" layer="96" ratio="10" rot="SR0"/>
+<attribute name="NAME" x="106.2228" y="126.0094" size="3.4798" layer="95" ratio="10" rot="SR0"/>
+<attribute name="C3" x="106.68" y="119.38" size="1.778" layer="96"/>
 </instance>
 <instance part="TP1" gate="G$1" x="312.42" y="226.06" smashed="yes">
@@
 <label x="304.8" y="180.34" size="1.778" layer="95"/>
 </segment>
+<segment>
+<pinref part="C1" gate="A" pin="2"/>
+<wire x1="53.34" y1="119.38" x2="53.34" y2="101.6" width="0.1524" layer="91"/>
+<pinref part="C3" gate="A" pin="2"/>
+<wire x1="53.34" y1="101.6" x2="76.2" y2="101.6" width="0.1524" layer="91"/>
+<wire x1="76.2" y1="101.6" x2="104.14" y2="101.6" width="0.1524" layer="91"/>
+<wire x1="104.14" y1="101.6" x2="104.14" y2="119.38" width="0.1524" layer="91"/>
+<pinref part="C2" gate="A" pin="2"/>
+<wire x1="76.2" y1="119.38" x2="76.2" y2="101.6" width="0.1524" layer="91"/>
+<junction x="76.2" y="101.6"/>
+<wire x1="76.2" y1="101.6" x2="76.2" y2="93.98" width="0.1524" layer="91"/>
+<label x="76.2" y="93.98" size="1.778" layer="95"/>
+</segment>
 </net>
 <net name="12V" class="0">
@@
 </segment>
 <segment>
-<pinref part="C1" gate="A" pin="2"/>
-<wire x1="78.74" y1="129.54" x2="119.38" y2="129.54" width="0.1524" layer="91"/>
-<pinref part="C3" gate="A" pin="2"/>
-<wire x1="119.38" y1="129.54" x2="119.38" y2="106.68" width="0.1524" layer="91"/>
-<wire x1="119.38" y1="106.68" x2="119.38" y2="83.82" width="0.1524" layer="91"/>
-<wire x1="119.38" y1="83.82" x2="78.74" y2="83.82" width="0.1524" layer="91"/>
-<pinref part="C2" gate="A" pin="2"/>
-<wire x1="78.74" y1="106.68" x2="119.38" y2="106.68" width="0.1524" layer="91"/>
-<junction x="119.38" y="106.68"/>
-<wire x1="119.38" y1="106.68" x2="137.16" y2="106.68" width="0.1524" layer="91"/>
-<label x="137.16" y="106.68" size="1.778" layer="95"/>
-</segment>
-<segment>
 <pinref part="TP1" gate="G$1" pin="1"/>
 <wire x1="312.42" y1="226.06" x2="304.8" y2="226.06" width="0.1524" layer="91"/>
 <label x="304.8" y="226.06" size="1.778" layer="95"/>
 </segment>
+<segment>
+<pinref part="C1" gate="A" pin="1"/>
+<wire x1="53.34" y1="127" x2="53.34" y2="139.7" width="0.1524" layer="91"/>
+<pinref part="C3" gate="A" pin="1"/>
+<wire x1="53.34" y1="139.7" x2="76.2" y2="139.7" width="0.1524" layer="91"/>
+<wire x1="76.2" y1="139.7" x2="104.14" y2="139.7" width="0.1524" layer="91"/>
+<wire x1="104.14" y1="139.7" x2="104.14" y2="127" width="0.1524" layer="91"/>
+<pinref part="C2" gate="A" pin="1"/>
+<wire x1="76.2" y1="127" x2="76.2" y2="139.7" width="0.1524" layer="91"/>
+<junction x="76.2" y="139.7"/>
+<wire x1="76.2" y1="139.7" x2="76.2" y2="149.86" width="0.1524" layer="91"/>
+<label x="76.2" y="149.86" size="1.778" layer="95"/>
+</segment>
 </net>
 <net name="N$2" class="0">
@@
 </segment>
 </net>
-<net name="12V_GND" class="0">
-<segment>
-<pinref part="C1" gate="A" pin="1"/>
-<wire x1="71.12" y1="129.54" x2="48.26" y2="129.54" width="0.1524" layer="91"/>
-<pinref part="C3" gate="A" pin="1"/>
-<wire x1="48.26" y1="129.54" x2="48.26" y2="106.68" width="0.1524" layer="91"/>
-<wire x1="48.26" y1="106.68" x2="48.26" y2="83.82" width="0.1524" layer="91"/>
-<wire x1="48.26" y1="83.82" x2="71.12" y2="83.82" width="0.1524" layer="91"/>
-<pinref part="C2" gate="A" pin="1"/>
-<wire x1="71.12" y1="106.68" x2="48.26" y2="106.68" width="0.1524" layer="91"/>
-<junction x="48.26" y="106.68"/>
-<wire x1="48.26" y1="106.68" x2="35.56" y2="106.68" width="0.1524" layer="91"/>
-<label x="35.56" y="106.68" size="1.778" layer="95" rot="R180"/>
-</segment>
-</net>

Commit message: Add files via upload
Connections:
- new net GPIO5: J3.9, U2.IN5
- new net GPIO6: J3.5, U2.IN6
- new net GPIO7: J3.10, U2.IN7
- new net GPIO8: J3.12
- new net SOL5_1: J1.4, U2.OUT5
- new net SOL6_1: J1.3, U2.OUT6
- new net SOL7_1: U2.OUT7
- net DGND: no longer J3.9
- net SOL1_1: now also J1.8; no longer J1.3
- net SOL2_1: now also J1.7; no longer J1.4
- net SOL3_1: now also J1.6; no longer J1.5
- net SOL4_1: now also J1.5; no longer J1.6

Commit message: Add files via upload
Connections:
- removed net DGND: J2.18
- net GND: now also J2.18, U2.GND
Changed lines of the file:
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@@
 <label x="299.72" y="205.74" size="1.778" layer="95"/>
+</segment>
+<segment>
+<pinref part="U2" gate="G$1" pin="GND"/>
+<wire x1="109.22" y1="38.1" x2="109.22" y2="33.02" width="0.1524" layer="91"/>
+<label x="109.22" y="33.02" size="1.778" layer="95"/>
+</segment>
+<segment>
+<pinref part="J2" gate="G$1" pin="18"/>
+<wire x1="312.42" y1="83.82" x2="320.04" y2="83.82" width="0.1524" layer="91"/>
+<label x="320.04" y="83.82" size="1.778" layer="95"/>
 </segment>
 </net>
@@
 </segment>
 </net>
-<net name="DGND" class="0">
-<segment>
-<pinref part="J2" gate="G$1" pin="18"/>
-<wire x1="312.42" y1="83.82" x2="320.04" y2="83.82" width="0.1524" layer="91"/>
-<label x="320.04" y="83.82" size="1.778" layer="95"/>
-</segment>
-</net>

Commit message: Add files via upload
Parts:
- removed D1, D2: HLMP6, display-hp:HLMP6
- removed TP1, TP2, TP3, TP4, TP5, TP6, TP7: TEST-POINT3, SparkFun-Connectors:TEST-POINT3
- added D3, D4: (no value), SparkFun-LED:LED-GREEN0805-PG
- added J10, J11, J5, J6, J7, J8, J9: (no value), SparkFun-Connectors:CONN_01
- added J12, J13: 282837-3, X16_Backplane:282837-3
- J3: value SAMTEC-HTST-110-04-X-D-RAJ -> HTST-110-04-L-D-RA; device X16_Backplane:SAMTEC-HTST-110-04-X-D-RAJ -> X16_Backplane:HTST-110-04-L-D-RA
Connections:
- new net CLK: J3.9
- net 12V: now also D4.A, J12.1, J13.1, J5.1; no longer D1.A, TP1.1
- net 12V_GND: now also C1.2, C2.2, C3.2
- net 5V: now also D3.A, J3.20, J6.1; no longer D2.A, J3.1, TP2.1
- net CS: now also J11.1, J3.7; no longer J3.20, TP7.1
- net CTRL: now also J3.16; no longer J3.7
- net GND: now also J12.3, J13.3, J3.4, J7.1; no longer C1.2, C2.2, C3.2, J3.3, TP3.1
- net GPIO1: now also J3.1; no longer J3.2
- net GPIO2: now also J3.13; no longer J3.4
- net GPIO3: now also J3.14; no longer J3.6
- net GPIO4: now also J3.10; no longer J3.8
- net GPIO5: now also J3.8; no longer J3.9
- net GPIO6: now also J3.6; no longer J3.5
- net GPIO7: now also J3.5; no longer J3.10
- net GPIO8: now also J3.18; no longer J3.12
- net MISO: now also J3.12, J8.1; no longer J3.14, TP4.1
- net MOSI: now also J3.11, J9.1; no longer J3.16, TP5.1
- net N$2: now also D4.C; no longer D1.K
- net N$5: now also D3.C; no longer D2.K
- net PWMC0: now also J12.2
- net PWMC1: now also J13.2
- net SA0: now also J3.2; no longer J3.17
- net SA1: now also J3.15; no longer J3.19
- net SALERT: now also J3.3; no longer J3.13
- net SCL: now also J3.17; no longer J3.15
- net SCLK: now also J10.1; no longer J3.18, TP6.1
- net SDA: now also J3.19; no longer J3.11

Commit message: Add files via upload
Connections:
- removed net CLK: J3.9
- net SCLK: now also J3.9
Changed lines of the file:
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@@
 <label x="259.08" y="193.04" size="1.778" layer="95" rot="R180"/>
+</segment>
+<segment>
+<pinref part="J3" gate="A" pin="9"/>
+<wire x1="200.66" y1="71.12" x2="190.5" y2="71.12" width="0.1524" layer="91"/>
+<label x="190.5" y="71.12" size="1.778" layer="95"/>
 </segment>
 </net>
@@
 </segment>
 </net>
-<net name="CLK" class="0">
-<segment>
-<pinref part="J3" gate="A" pin="9"/>
-<wire x1="200.66" y1="71.12" x2="190.5" y2="71.12" width="0.1524" layer="91"/>
-<label x="190.5" y="71.12" size="1.778" layer="95"/>
-</segment>
-</net>

Commit message: Add files via upload
Parts:
- removed J5, J6, J7: (no value), SparkFun-Connectors:CONN_01
- added H1, H2, H3, H4: 6-32-HOLE, X16-ExtraComponents:6-32-HOLE
- added TP1, TP2, TP3, TP4: TESTPOINT_5.04MM, X16_Backplane:TESTPOINT_5.04MM
- U$1, U$2, U$3: value CONN_BACKPLANE_ESC_ADAPTER -> CONN_BACKPLANE_ESC_ADAPTER_NEW; device X16_Backplane:CONN_BACKPLANE_ESC_ADAPTER -> X16_Backplane:CONN_BACKPLANE_ESC_ADAPTER_NEW
Connections:
- net 12V: now also TP1.TP; no longer J5.1
- net 12V_GND: now also J12.3, J13.3, R1.1, TP2.TP
- net 12V_L: now also J2.08, J2.16, J2.24
- net 5V: now also TP3.TP; no longer J6.1
- net GND: now also TP4.TP, U$1.NC, U$2.NC, U$3.NC; no longer J12.3, J13.3, J7.1, R1.1
Other:
- moved on the sheet: J10, J11, J8, J9
