File: X16-Backplane1.sch (EAGLE design)
At the start: 29 parts, among them J1 CONN_PXC-8-RA-1778683, J12 282837-3, J13 282837-3, J2 CONN_ET60S-D04-3-08-D04-X-R1-S, J3 HTST-110-04-L-D-RA, J4 CLT-110-01-F-D, U2 TRANS_ULN2003AD

Commit message: Minh Update 1
Connections:
- net PWMC0: now also J13.2; no longer J12.2
- net PWMC1: now also J12.2; no longer J13.2
Changed lines of the file:
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@@
-</segment>
-</net>
-<net name="PWMC0" class="0">
-<segment>
-<pinref part="J12" gate="G$1" pin="2"/>
-<wire x1="203.2" y1="215.9" x2="195.58" y2="215.9" width="0.1524" layer="91"/>
-<label x="195.58" y="215.9" size="1.778" layer="95"/>
-</segment>
-</net>
-<net name="PWMC1" class="0">
-<segment>
-<pinref part="J13" gate="G$1" pin="2"/>
-<wire x1="203.2" y1="190.5" x2="195.58" y2="190.5" width="0.1524" layer="91"/>
-<label x="195.58" y="190.5" size="1.778" layer="95"/>
 </segment>
 </net>
@@
 </segment>
 </net>
+<net name="PWMC1" class="0">
+<segment>
+<pinref part="J12" gate="G$1" pin="2"/>
+<wire x1="203.2" y1="215.9" x2="195.58" y2="215.9" width="0.1524" layer="91"/>
+<label x="195.58" y="215.9" size="1.778" layer="95"/>
+</segment>
+</net>
+<net name="PWMC0" class="0">
+<segment>
+<pinref part="J13" gate="G$1" pin="2"/>
+<wire x1="203.2" y1="190.5" x2="195.58" y2="190.5" width="0.1524" layer="91"/>
+<label x="195.58" y="190.5" size="1.778" layer="95"/>
+</segment>
+</net>

Commit message: Minh Update 3
Parts:
- removed J10, J11, J8, J9: (no value), SparkFun-Connectors:CONN_01
- added JP1: (no value), X16-ExtraComponents:TEST_PIN-1X4
Connections:
- net CS: now also JP1.4; no longer J11.1
- net MISO: now also JP1.1; no longer J8.1
- net MOSI: now also JP1.2; no longer J9.1
- net SCLK: now also JP1.3; no longer J10.1
Changed lines of the file:
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@@
 <part name="J3" library="X16_Backplane" deviceset="HTST-110-04-L-D-RA" device=""/>
 <part name="J4" library="X16_Backplane" deviceset="CLT-110-01-F-D" device=""/>
-<part name="J8" library="SparkFun-Connectors" library_urn="urn:adsk.eagle:library:513" deviceset="CONN_01" device="" package3d_urn="urn:adsk.eagle:package:38028/2"/>
-<part name="J9" library="SparkFun-Connectors" library_urn="urn:adsk.eagle:library:513" deviceset="CONN_01" device="" package3d_urn="urn:adsk.eagle:package:38028/2"/>
-<part name="J10" library="SparkFun-Connectors" library_urn="urn:adsk.eagle:library:513" deviceset="CONN_01" device="" package3d_urn="urn:adsk.eagle:package:38028/2"/>
-<part name="J11" library="SparkFun-Connectors" library_urn="urn:adsk.eagle:library:513" deviceset="CONN_01" device="" package3d_urn="urn:adsk.eagle:package:38028/2"/>
 <part name="J12" library="X16_Backplane" deviceset="282837-3" device=""/>
 <part name="J13" library="X16_Backplane" deviceset="282837-3" device=""/>
@@
 <part name="H3" library="X16-ExtraComponents" deviceset="6-32-HOLE" device=""/>
 <part name="H4" library="X16-ExtraComponents" deviceset="6-32-HOLE" device=""/>
+<part name="JP1" library="X16-ExtraComponents" deviceset="TEST_PIN-1X4" device="" package3d_urn="urn:adsk.eagle:package:22407/2"/>
 </parts>
 <sheets>
@@
 <attribute name="C3" x="106.68" y="119.38" size="1.778" layer="96"/>
 </instance>
-<instance part="J8" gate="J1" x="304.8" y="129.54" smashed="yes">
-<attribute name="VALUE" x="302.26" y="124.714" size="1.778" layer="96" font="vector"/>
-<attribute name="NAME" x="302.26" y="132.588" size="1.778" layer="95" font="vector"/>
-</instance>
-<instance part="J9" gate="J1" x="304.8" y="104.14" smashed="yes">
-<attribute name="VALUE" x="302.26" y="99.314" size="1.778" layer="96" font="vector"/>
-<attribute name="NAME" x="302.26" y="107.188" size="1.778" layer="95" font="vector"/>
-</instance>
-<instance part="J10" gate="J1" x="304.8" y="83.82" smashed="yes">
-<attribute name="VALUE" x="302.26" y="78.994" size="1.778" layer="96" font="vector"/>
-<attribute name="NAME" x="302.26" y="86.868" size="1.778" layer="95" font="vector"/>
-</instance>
-<instance part="J11" gate="J1" x="304.8" y="66.04" smashed="yes">
-<attribute name="VALUE" x="302.26" y="61.214" size="1.778" layer="96" font="vector"/>
-<attribute name="NAME" x="302.26" y="69.088" size="1.778" layer="95" font="vector"/>
-</instance>
 <instance part="J12" gate="G$1" x="210.82" y="215.9" smashed="yes">
 <attribute name="NAME" x="207.769640625" y="221.49233125" size="1.27098125" layer="95"/>
@@
 <attribute name="NAME" x="256.54" y="165.1" size="1.016" layer="95" align="bottom-center"/>
 <attribute name="VALUE" x="256.54" y="160.02" size="1.016" layer="95" align="top-center"/>
+</instance>
+<instance part="JP1" gate="A" x="353.06" y="121.92" smashed="yes">
+<attribute name="NAME" x="346.71" y="130.175" size="1.778" layer="95"/>
+<attribute name="VALUE" x="346.71" y="114.3" size="1.778" layer="96"/>
 </instance>
 </instances>
@@
 </segment>
 </net>
-<net name="MISO" class="0">
-<segment>
-<pinref part="J8" gate="J1" pin="1"/>
-<wire x1="312.42" y1="129.54" x2="320.04" y2="129.54" width="0.1524" layer="91"/>
-<label x="320.04" y="129.54" size="1.778" layer="95"/>
-</segment>
-</net>
-<net name="MOSI" class="0">
-<segment>
-<pinref part="J9" gate="J1" pin="1"/>
-<wire x1="312.42" y1="104.14" x2="320.04" y2="104.14" width="0.1524" layer="91"/>
-<label x="320.04" y="104.14" size="1.778" layer="95"/>
-</segment>
-</net>
-<net name="SCLK" class="0">
-<segment>
-<pinref part="J10" gate="J1" pin="1"/>
-<wire x1="312.42" y1="83.82" x2="320.04" y2="83.82" width="0.1524" layer="91"/>
-<label x="320.04" y="83.82" size="1.778" layer="95"/>
-</segment>
-</net>
-<net name="CS" class="0">
-<segment>
-<pinref part="J11" gate="J1" pin="1"/>
-<wire x1="312.42" y1="66.04" x2="320.04" y2="66.04" width="0.1524" layer="91"/>
-<label x="320.04" y="66.04" size="1.778" layer="95"/>
-</segment>
-</net>
 <net name="12V_GND" class="0">
 <segment>
@@
 </segment>
 </net>
+<net name="MISO" class="0">
+<segment>
+<wire x1="347.98" y1="127" x2="335.28" y2="127" width="0.1524" layer="91"/>
+<label x="335.28" y="127" size="1.778" layer="95"/>
+<pinref part="JP1" gate="A" pin="1"/>
+</segment>
+</net>
+<net name="MOSI" class="0">
+<segment>
+<wire x1="347.98" y1="124.46" x2="335.28" y2="124.46" width="0.1524" layer="91"/>
+<label x="335.28" y="124.46" size="1.778" layer="95"/>
+<pinref part="JP1" gate="A" pin="2"/>
+</segment>
+</net>
+<net name="SCLK" class="0">
+<segment>
+<wire x1="347.98" y1="121.92" x2="335.28" y2="121.92" width="0.1524" layer="91"/>
+<label x="335.28" y="121.92" size="1.778" layer="95"/>
+<pinref part="JP1" gate="A" pin="3"/>
+</segment>
+</net>
+<net name="CS" class="0">
+<segment>
+<wire x1="347.98" y1="119.38" x2="335.28" y2="119.38" width="0.1524" layer="91"/>
+<label x="335.28" y="119.38" size="1.778" layer="95"/>
+<pinref part="JP1" gate="A" pin="4"/>
+</segment>
+</net>

Commit message: Minh Update 5
Parts:
- D3, D4: device SparkFun-LED:LED-GREEN0805-PG -> led:LEDCHIPLED_0805
- H1, H2, H3, H4: device X16-ExtraComponents:6-32-HOLE -> X16_Backplane:6-32-HOLE
Connections:
- removed net SA0: J2.22, J3.2
- removed net SA1: J2.23, J3.15
Changed lines of the file:
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@@
 <part name="J2" library="X16_Backplane" deviceset="CONN_ET60S-D04-3-08-D04-X-R1-S" device=""/>
 <part name="FRAME2" library="frames" library_urn="urn:adsk.eagle:library:229" deviceset="A3L-LOC" device=""/>
-<part name="R1" library="SparkFun-Resistors" library_urn="urn:adsk.eagle:library:532" deviceset="RESISTOR" device="0603" package3d_urn="urn:adsk.eagle:package:41389018/1" value=" ">
+<part name="R1" library="SparkFun-Resistors" library_urn="urn:adsk.eagle:library:532" deviceset="RESISTOR" device="0603" package3d_urn="urn:adsk.eagle:package:39650/1" value=" ">
 <attribute name="PROD_ID" value="600"/>
 </part>
-<part name="R2" library="SparkFun-Resistors" library_urn="urn:adsk.eagle:library:532" deviceset="RESISTOR" device="0603" package3d_urn="urn:adsk.eagle:package:41389018/1" value=" ">
+<part name="R2" library="SparkFun-Resistors" library_urn="urn:adsk.eagle:library:532" deviceset="RESISTOR" device="0603" package3d_urn="urn:adsk.eagle:package:39650/1" value=" ">
 <attribute name="PROD_ID" value="250"/>
 </part>
@@
 <part name="J12" library="X16_Backplane" deviceset="282837-3" device=""/>
 <part name="J13" library="X16_Backplane" deviceset="282837-3" device=""/>
-<part name="D3" library="SparkFun-LED" library_urn="urn:adsk.eagle:library:529" deviceset="LED-GREEN" device="0805-PG" package3d_urn="urn:adsk.eagle:package:41389318/1"/>
-<part name="D4" library="SparkFun-LED" library_urn="urn:adsk.eagle:library:529" deviceset="LED-GREEN" device="0805-PG" package3d_urn="urn:adsk.eagle:package:41389318/1"/>
+<part name="D3" library="led" library_urn="urn:adsk.eagle:library:259" deviceset="LED" device="CHIPLED_0805" package3d_urn="urn:adsk.eagle:package:15821/2"/>
+<part name="D4" library="led" library_urn="urn:adsk.eagle:library:259" deviceset="LED" device="CHIPLED_0805" package3d_urn="urn:adsk.eagle:package:15821/2"/>
 <part name="TP1" library="X16_Backplane" deviceset="TESTPOINT_5.04MM" device=""/>
 <part name="TP2" library="X16_Backplane" deviceset="TESTPOINT_5.04MM" device=""/>
 <part name="TP3" library="X16_Backplane" deviceset="TESTPOINT_5.04MM" device=""/>
 <part name="TP4" library="X16_Backplane" deviceset="TESTPOINT_5.04MM" device=""/>
-<part name="H1" library="X16-ExtraComponents" deviceset="6-32-HOLE" device=""/>
-<part name="H2" library="X16-ExtraComponents" deviceset="6-32-HOLE" device=""/>
-<part name="H3" library="X16-ExtraComponents" deviceset="6-32-HOLE" device=""/>
-<part name="H4" library="X16-ExtraComponents" deviceset="6-32-HOLE" device=""/>
+<part name="H1" library="X16_Backplane" deviceset="6-32-HOLE" device=""/>
+<part name="H2" library="X16_Backplane" deviceset="6-32-HOLE" device=""/>
+<part name="H3" library="X16_Backplane" deviceset="6-32-HOLE" device=""/>
+<part name="H4" library="X16_Backplane" deviceset="6-32-HOLE" device=""/>
 <part name="JP1" library="X16-ExtraComponents" deviceset="TEST_PIN-1X4" device="" package3d_urn="urn:adsk.eagle:package:22407/2"/>
 </parts>
@@
 </segment>
 </net>
-<net name="SA0" class="0">
-<segment>
-<pinref part="J2" gate="G$1" pin="22"/>
-<wire x1="312.42" y1="73.66" x2="320.04" y2="73.66" width="0.1524" layer="91"/>
-<label x="320.04" y="73.66" size="1.778" layer="95"/>
-</segment>
-<segment>
-<pinref part="J3" gate="A" pin="2"/>
-<wire x1="200.66" y1="88.9" x2="190.5" y2="88.9" width="0.1524" layer="91"/>
-<label x="190.5" y="88.9" size="1.778" layer="95"/>
-</segment>
-</net>
-<net name="SA1" class="0">
-<segment>
-<pinref part="J2" gate="G$1" pin="23"/>
-<wire x1="312.42" y1="71.12" x2="320.04" y2="71.12" width="0.1524" layer="91"/>
-<label x="320.04" y="71.12" size="1.778" layer="95"/>
-</segment>
-<segment>
-<pinref part="J3" gate="A" pin="15"/>
-<wire x1="200.66" y1="55.88" x2="190.5" y2="55.88" width="0.1524" layer="91"/>
-<label x="190.5" y="55.88" size="1.778" layer="95"/>
-</segment>
-</net>

Commit message: Minh Update 6
Parts:
- added ESC_JP1, ESC_JP2, SERVO_JP1, SERVO_JP2: (no value), X16-ExtraComponents:TEST_PIN-1X2
Connections:
- new net N$1: ESC_JP1.1, U$3.PWM0
- new net N$3: ESC_JP2.1, U$3.PWM1
- new net PWMC0_CONN: J13.2, SERVO_JP1.2
- new net PWMC1_CONN: J12.2, SERVO_JP2.2
- net CTRL: now also J2.23; no longer J2.17
- net GND: now also J2.22; no longer J2.18
- net PWMC0: now also ESC_JP1.2, SERVO_JP1.1; no longer J13.2, U$3.PWM0
- net PWMC1: now also ESC_JP2.2, SERVO_JP2.1; no longer J12.2, U$3.PWM1
- net SCL: now also J2.19; no longer J2.21
- net SDA: now also J2.21; no longer J2.19
Changed lines of the file:
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@@
 <part name="H4" library="X16_Backplane" deviceset="6-32-HOLE" device=""/>
 <part name="JP1" library="X16-ExtraComponents" deviceset="TEST_PIN-1X4" device="" package3d_urn="urn:adsk.eagle:package:22407/2"/>
+<part name="SERVO_JP2" library="X16-ExtraComponents" deviceset="TEST_PIN-1X2" device="" package3d_urn="urn:adsk.eagle:package:22435/2"/>
+<part name="SERVO_JP1" library="X16-ExtraComponents" deviceset="TEST_PIN-1X2" device="" package3d_urn="urn:adsk.eagle:package:22435/2"/>
+<part name="ESC_JP1" library="X16-ExtraComponents" deviceset="TEST_PIN-1X2" device="" package3d_urn="urn:adsk.eagle:package:22435/2"/>
+<part name="ESC_JP2" library="X16-ExtraComponents" deviceset="TEST_PIN-1X2" device="" package3d_urn="urn:adsk.eagle:package:22435/2"/>
 </parts>
 <sheets>
@@
 <attribute name="VALUE" x="271.78" y="175.26" size="1.778" layer="96"/>
 </instance>
+<instance part="ESC_JP1" gate="G$1" x="223.52" y="187.96" smashed="yes">
+<attribute name="NAME" x="217.17" y="193.675" size="1.778" layer="95"/>
+<attribute name="VALUE" x="217.17" y="182.88" size="1.778" layer="96"/>
+</instance>
+<instance part="ESC_JP2" gate="G$1" x="223.52" y="175.26" smashed="yes">
+<attribute name="NAME" x="217.17" y="180.975" size="1.778" layer="95"/>
+<attribute name="VALUE" x="217.17" y="170.18" size="1.778" layer="96"/>
+</instance>
 </instances>
 <busses>
@@
 <net name="PWMC0" class="0">
 <segment>
-<pinref part="U$3" gate="G$1" pin="PWM0"/>
-<wire x1="175.26" y1="190.5" x2="182.88" y2="190.5" width="0.1524" layer="91"/>
-<label x="182.88" y="190.5" size="1.778" layer="95"/>
-</segment>
-<segment>
 <pinref part="J4" gate="G$1" pin="14"/>
 <wire x1="292.1" y1="187.96" x2="299.72" y2="187.96" width="0.1524" layer="91"/>
 <label x="299.72" y="187.96" size="1.778" layer="95"/>
 </segment>
+<segment>
+<wire x1="218.44" y1="187.96" x2="210.82" y2="187.96" width="0.1524" layer="91"/>
+<label x="210.82" y="187.96" size="1.778" layer="95" rot="MR0"/>
+<pinref part="ESC_JP1" gate="G$1" pin="2"/>
+</segment>
 </net>
 <net name="PWMC1" class="0">
-<segment>
-<pinref part="U$3" gate="G$1" pin="PWM1"/>
-<wire x1="175.26" y1="187.96" x2="182.88" y2="187.96" width="0.1524" layer="91"/>
-<label x="182.88" y="187.96" size="1.778" layer="95"/>
-</segment>
 <segment>
 <pinref part="J4" gate="G$1" pin="16"/>
 <wire x1="292.1" y1="185.42" x2="299.72" y2="185.42" width="0.1524" layer="91"/>
 <label x="299.72" y="185.42" size="1.778" layer="95"/>
+</segment>
+<segment>
+<wire x1="218.44" y1="175.26" x2="210.82" y2="175.26" width="0.1524" layer="91"/>
+<label x="210.82" y="175.26" size="1.778" layer="95" rot="MR0"/>
+<pinref part="ESC_JP2" gate="G$1" pin="2"/>
 </segment>
 </net>
@@
 </segment>
 <segment>
-<pinref part="J2" gate="G$1" pin="18"/>
-<wire x1="312.42" y1="83.82" x2="320.04" y2="83.82" width="0.1524" layer="91"/>
-<label x="320.04" y="83.82" size="1.778" layer="95"/>
-</segment>
-<segment>
 <pinref part="J3" gate="A" pin="4"/>
 <wire x1="200.66" y1="83.82" x2="190.5" y2="83.82" width="0.1524" layer="91"/>
@@
 <wire x1="175.26" y1="180.34" x2="182.88" y2="180.34" width="0.1524" layer="91"/>
 <label x="182.88" y="180.34" size="1.778" layer="95"/>
+</segment>
+<segment>
+<wire x1="312.42" y1="73.66" x2="320.04" y2="73.66" width="0.1524" layer="91"/>
+<label x="320.04" y="73.66" size="1.778" layer="95"/>
+<pinref part="J2" gate="G$1" pin="22"/>
 </segment>
 </net>
@@
 <net name="CTRL" class="0">
 <segment>
-<pinref part="J2" gate="G$1" pin="17"/>
-<wire x1="312.42" y1="86.36" x2="320.04" y2="86.36" width="0.1524" layer="91"/>
-<label x="320.04" y="86.36" size="1.778" layer="95"/>
-</segment>
-<segment>
 <pinref part="J3" gate="A" pin="16"/>
 <wire x1="200.66" y1="53.34" x2="190.5" y2="53.34" width="0.1524" layer="91"/>
 <label x="190.5" y="53.34" size="1.778" layer="95"/>
 </segment>
+<segment>
+<wire x1="312.42" y1="71.12" x2="320.04" y2="71.12" width="0.1524" layer="91"/>
+<label x="320.04" y="71.12" size="1.778" layer="95"/>
+<pinref part="J2" gate="G$1" pin="23"/>
+</segment>
 </net>
 <net name="SDA" class="0">
-<segment>
-<pinref part="J2" gate="G$1" pin="19"/>
-<wire x1="312.42" y1="81.28" x2="320.04" y2="81.28" width="0.1524" layer="91"/>
-<label x="320.04" y="81.28" size="1.778" layer="95"/>
-</segment>
 <segment>
 <pinref part="J3" gate="A" pin="19"/>
@@
 <label x="190.5" y="45.72" size="1.778" layer="95"/>
 </segment>
+<segment>
+<wire x1="312.42" y1="76.2" x2="320.04" y2="76.2" width="0.1524" layer="91"/>
+<label x="320.04" y="76.2" size="1.778" layer="95"/>
+<pinref part="J2" gate="G$1" pin="21"/>
+</segment>
 </net>
 <net name="SALERT" class="0">
-<segment>
-<pinref part="J2" gate="G$1" pin="20"/>
-<wire x1="312.42" y1="78.74" x2="320.04" y2="78.74" width="0.1524" layer="91"/>
-<label x="320.04" y="78.74" size="1.778" layer="95"/>
-</segment>
 <segment>
 <pinref part="J3" gate="A" pin="3"/>
@@
 <label x="190.5" y="86.36" size="1.778" layer="95"/>
 </segment>
+<segment>
+<wire x1="312.42" y1="78.74" x2="320.04" y2="78.74" width="0.1524" layer="91"/>
+<label x="320.04" y="78.74" size="1.778" layer="95"/>
+<pinref part="J2" gate="G$1" pin="20"/>
+</segment>
 </net>
 <net name="SCL" class="0">
-<segment>
-<pinref part="J2" gate="G$1" pin="21"/>
-<wire x1="312.42" y1="76.2" x2="320.04" y2="76.2" width="0.1524" layer="91"/>
-<label x="320.04" y="76.2" size="1.778" layer="95"/>
-</segment>
 <segment>
 <pinref part="J3" gate="A" pin="17"/>
@@
 <label x="190.5" y="50.8" size="1.778" layer="95"/>
 </segment>
+<segment>
+<wire x1="312.42" y1="81.28" x2="320.04" y2="81.28" width="0.1524" layer="91"/>
+<label x="320.04" y="81.28" size="1.778" layer="95"/>
+<pinref part="J2" gate="G$1" pin="19"/>
+</segment>
 </net>
 <net name="GPIO1" class="0">
@@
 <wire x1="200.66" y1="48.26" x2="190.5" y2="48.26" width="0.1524" layer="91"/>
 <label x="190.5" y="48.26" size="1.778" layer="95"/>
+</segment>
+</net>
+<net name="N$1" class="0">
+<segment>
+<pinref part="ESC_JP1" gate="G$1" pin="1"/>
+<pinref part="U$3" gate="G$1" pin="PWM0"/>
+<wire x1="218.44" y1="190.5" x2="175.26" y2="190.5" width="0.1524" layer="91"/>
+</segment>
+</net>
+<net name="N$3" class="0">
+<segment>
+<pinref part="ESC_JP2" gate="G$1" pin="1"/>
+<wire x1="218.44" y1="177.8" x2="198.12" y2="177.8" width="0.1524" layer="91"/>
+<wire x1="198.12" y1="177.8" x2="198.12" y2="187.96" width="0.1524" layer="91"/>
+<pinref part="U$3" gate="G$1" pin="PWM1"/>
+<wire x1="198.12" y1="187.96" x2="175.26" y2="187.96" width="0.1524" layer="91"/>
 </segment>
 </net>
@@
 <attribute name="VALUE" x="346.71" y="114.3" size="1.778" layer="96"/>
 </instance>
+<instance part="SERVO_JP2" gate="G$1" x="228.6" y="215.9" smashed="yes">
+<attribute name="NAME" x="222.25" y="221.615" size="1.778" layer="95"/>
+<attribute name="VALUE" x="222.25" y="210.82" size="1.778" layer="96"/>
+</instance>
+<instance part="SERVO_JP1" gate="G$1" x="228.6" y="190.5" smashed="yes">
+<attribute name="NAME" x="222.25" y="196.215" size="1.778" layer="95"/>
+<attribute name="VALUE" x="222.25" y="185.42" size="1.778" layer="96"/>
+</instance>
 </instances>
 <busses>
@@
 </segment>
 </net>
-<net name="PWMC1" class="0">
-<segment>
-<pinref part="J12" gate="G$1" pin="2"/>
-<wire x1="203.2" y1="215.9" x2="195.58" y2="215.9" width="0.1524" layer="91"/>
-<label x="195.58" y="215.9" size="1.778" layer="95"/>
-</segment>
-</net>
-<net name="PWMC0" class="0">
-<segment>
-<pinref part="J13" gate="G$1" pin="2"/>
-<wire x1="203.2" y1="190.5" x2="195.58" y2="190.5" width="0.1524" layer="91"/>
-<label x="195.58" y="190.5" size="1.778" layer="95"/>
-</segment>
-</net>
 <net name="MISO" class="0">
 <segment>
@@
 </segment>
 </net>
+<net name="PWMC1" class="0">
+<segment>
+<wire x1="223.52" y1="218.44" x2="215.9" y2="218.44" width="0.1524" layer="91"/>
+<label x="215.9" y="218.44" size="1.778" layer="95"/>
+<pinref part="SERVO_JP2" gate="G$1" pin="1"/>
+</segment>
+</net>
+<net name="PWMC1_CONN" class="0">
+<segment>
+<pinref part="SERVO_JP2" gate="G$1" pin="2"/>
+<wire x1="223.52" y1="215.9" x2="215.9" y2="215.9" width="0.1524" layer="91"/>
+<label x="215.9" y="215.9" size="1.778" layer="95"/>
+</segment>
+<segment>
+<wire x1="203.2" y1="215.9" x2="195.58" y2="215.9" width="0.1524" layer="91"/>
+<label x="195.58" y="215.9" size="1.778" layer="95"/>
+<pinref part="J12" gate="G$1" pin="2"/>
+</segment>
+</net>
+<net name="PWMC0" class="0">
+<segment>
+<wire x1="223.52" y1="193.04" x2="215.9" y2="193.04" width="0.1524" layer="91"/>
+<label x="215.9" y="193.04" size="1.778" layer="95"/>
+<pinref part="SERVO_JP1" gate="G$1" pin="1"/>
+</segment>
+</net>
+<net name="PWMC0_CONN" class="0">
+<segment>
+<pinref part="SERVO_JP1" gate="G$1" pin="2"/>
+<wire x1="223.52" y1="190.5" x2="215.9" y2="190.5" width="0.1524" layer="91"/>
+<label x="215.9" y="190.5" size="1.778" layer="95"/>
+</segment>
+<segment>
+<wire x1="203.2" y1="190.5" x2="195.58" y2="190.5" width="0.1524" layer="91"/>
+<label x="195.58" y="190.5" size="1.778" layer="95"/>
+<pinref part="J13" gate="G$1" pin="2"/>
+</segment>
+</net>

Commit message: GERBER file created
Connections:
- net GND renamed GNDRAT
Changed lines of the file:
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@@
 </segment>
 </net>
-<net name="GND" class="0">
+<net name="GNDRAT" class="0">
 <segment>
 <pinref part="J2" gate="G$1" pin="P06"/>
@@
 </segment>
 </net>
-<net name="GND" class="0">
+<net name="GNDRAT" class="0">
 <segment>
 <pinref part="R2" gate="G$1" pin="1"/>
